File: integrated/schematic/pantiltslide_integrated.kicad_pcb (KiCad board)
At the start: 4 copper layers, 150 x 120 mm, 80 parts, among them J1 24V_In, J10 Enc_Jog, J11 Enc_Angle, J12 Limit_Min, J13 Limit_Max, J14 Limit_Z_Home, J2 USB_PROG, J3 Motor_Slide, J4 Motor_Pan, J5 Motor_Tilt, J6 Motor_Z, J7 AS5600_Pan, J8 AS5600_Tilt, J9 OLED, SW1 BOOT, SW2 RESET, U1 LM2596S-5, U2 AMS1117-3.3, U3 ESP32-S3-WROOM-1-N16R8, U4 TMC2209-LA, U5 TMC2209-LA, U6 TMC2209-LA, U7 TMC2209-LA, U8 TCA9548APWR

Commit message: updates
Parts:
- J10, J11, J3, J4, J5, J6, J7, J8, J9: footprint Connector_PinHeader_2.54mm:PinHeader_1x04_P2.54mm_Vertical -> Connector_JST:JST_XH_B4B-XH-A_1x04_P2.50mm_Vertical
- J12, J13, J14: footprint TerminalBlock:TerminalBlock_Altech_AK300-2_P5.00mm -> Connector_JST:JST_XH_B2B-XH-A_1x02_P2.50mm_Vertical
- moved C10 115.9 mm to (146.9, 27.6)
- moved C15 98.0 mm to (94.9, 27.6)
- moved C20 87.0 mm to (133.9, 43.6)
- moved C25 58.5 mm to (94.9, 70.6)
- moved J11 55.6 mm to (26.3, 119.2)
- moved R3 55.0 mm to (155.9, 24.1)
- moved R4 55.0 mm to (159.9, 24.1)
- moved C30 40.0 mm to (133.9, 86.6)
- moved J3 38.8 mm to (95.3, 124.2)
- moved J7 34.8 mm to (26.3, 111.2)
- moved J4 28.8 mm to (110.3, 124.2)
- moved J8 24.8 mm to (41.3, 111.2)
- moved R20 22.0 mm to (53.9, 48.1)
- moved R21 22.0 mm to (57.9, 48.1)
- moved J5 18.9 mm to (125.3, 124.2)
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
Commit message: latest version
Parts:
- C10: footprint Capacitor_THT:CP_Radial_D8.0mm_P3.50mm -> Capacitor_SMD:C_0805_2012Metric
- moved C10 103.5 mm to (43.5, 33.0), turned to 90 degrees
- moved C2 51.3 mm to (24.5, 80.0)
- moved C4 46.4 mm to (41.2, 80.6)
- moved C5 43.2 mm to (45.8, 79.8)
- moved C9 34.2 mm to (43.5, 29.5), turned to 90 degrees
- moved C14 33.3 mm to (89.8, 27.3)
- moved C8 32.6 mm to (43.5, 26.0), turned to 90 degrees
- moved C7 31.8 mm to (43.5, 22.5), turned to 90 degrees
- moved R20 30.3 mm to (84.0, 45.3)
- moved C1 29.0 mm to (27.5, 99.5)
- moved C3 28.7 mm to (37.9, 100.1)
- moved C13 27.3 mm to (92.6, 31.7)
- moved C18 26.9 mm to (134.6, 53.7)
- moved R3 25.9 mm to (130.0, 23.3)
- moved R4 24.9 mm to (135.0, 23.3)
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Connections:
- net SW_NODE renamed /SW_NODE
- D2 pad 1: USB_VBUS -> +5V
- D2 pad 2: +5V -> USB_VBUS
- F1 pad 1: +24V -> /+24V_RAW
- J1 pad 1: +24V -> /+24V_RAW

Commit message: switching tmc2209s to new schmatic file
Parts:
- J1: footprint TerminalBlock:TerminalBlock_Altech_AK300-2_P5.00mm -> TerminalBlock:TerminalBlock_MaiXu_MX126-5.0-02P_1x02_P5.00mm
- moved C31 242.6 mm to (270.0, 84.3)
- moved U8 237.2 mm to (270.6, 92.5)
- moved R14 207.8 mm to (277.0, 89.7), turned to 90 degrees
- moved R15 204.7 mm to (278.9, 89.7), turned to 90 degrees
- moved J12 204.0 mm to (242.2, 91.2)
- moved J13 192.9 mm to (242.2, 99.0)
- moved R21 183.0 mm to (236.6, 60.3), turned to 90 degrees
- moved J14 181.9 mm to (242.2, 106.8)
- moved J9 179.5 mm to (229.1, 64.9)
- moved J7 176.5 mm to (197.8, 71.5)
- moved R16 160.1 mm to (200.8, 76.8), turned to 180 degrees
- moved J8 159.6 mm to (197.9, 82.4)
- moved R17 158.4 mm to (204.4, 67.3), turned to 180 degrees
- moved R18 150.9 mm to (200.6, 87.4), turned to 180 degrees
- moved R20 150.8 mm to (234.1, 60.3), turned to 90 degrees
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Connections:
- C12 pad 2: +24V -> Net-(C12-Pad2)
- C13 pad 2: GND -> unconnected-(C13-Pad2)
- C14 pad 1: +24V -> Net-(C12-Pad2)
- C15 pad 1: +24V -> Net-(C12-Pad2)
- C19 pad 2: GND -> unconnected-(C19-Pad2)
- C23 pad 1: 5VOUT_Tilt -> unconnected-(C23-Pad1)
- C23 pad 2: GND -> 5VOUT_Tilt
- C24 pad 1: +24V -> unconnected-(C24-Pad1)
- C24 pad 2: GND -> unconnected-(C24-Pad2)
- C25 pad 1: +24V -> unconnected-(C25-Pad1)
- C25 pad 2: GND -> +24V
- C28 pad 1: 5VOUT_Z -> unconnected-(C28-Pad1)
- C28 pad 2: GND -> 5VOUT_Z
- C29 pad 1: +24V -> unconnected-(C29-Pad1)
- C29 pad 2: GND -> unconnected-(C29-Pad2)
- C30 pad 1: +24V -> unconnected-(C30-Pad1)
- C30 pad 2: GND -> +24V
- D1 pad 1: /SW_NODE -> unconnected-(D1-K-Pad1)
- L1 pad 1: /SW_NODE -> +5V
- L1 pad 2: +5V -> GND
- U1 pad 2: /SW_NODE -> GND
- U4 pad 22: +24V -> Net-(C12-Pad2)
- U4 pad 28: +24V -> Net-(C12-Pad2)
Routing:
- net GND: track 0.00 -> 120.1 mm
- net +24V: track 0.00 -> 21.3 mm
- net +5V: track 0.00 -> 18.4 mm
- net +3V3: track 0.00 -> 15.8 mm
- net MOTOR_Slide_A2: track 0.00 -> 12.3 mm
- net MOTOR_Pan_A2: track 0.00 -> 8.74 mm, vias 0 -> 2
- net MOTOR_Pan_B2: track 0.00 -> 8.74 mm
- net MOTOR_Pan_A1: track 0.00 -> 8.60 mm
- net USBCC2: track 0.00 -> 8.57 mm
- net MOTOR_Pan_B1: track 0.00 -> 7.56 mm
- net /+24V_RAW: track 0.00 -> 6.96 mm
- net MOTOR_Slide_B2: track 0.00 -> 6.54 mm
- net USB_VBUS: track 0.00 -> 6.52 mm
- net MOTOR_Slide_A1: track 0.00 -> 6.40 mm
- net GPIO12: track 0.00 -> 6.15 mm
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
Commit message: integrated pcb steppers done
Parts:
- removed C10: 10uF, Capacitor_SMD:C_0805_2012Metric
- removed C17, C19, C22, C24, C27, C29, C31, C7, C8, C9: 100nF, Capacitor_SMD:C_0603_1608Metric
- removed C18, C23, C28: 4.7uF, Capacitor_SMD:C_0603_1608Metric
- removed C20, C25, C30: 100uF_35V, Capacitor_THT:CP_Radial_D8.0mm_P3.50mm
- removed C21, C26: 22nF, Capacitor_SMD:C_0603_1608Metric
- removed C6: 1uF, Capacitor_SMD:C_0603_1608Metric
- removed J10: Enc_Jog, Connector_JST:JST_XH_B4B-XH-A_1x04_P2.50mm_Vertical
- removed J11: Enc_Angle, Connector_JST:JST_XH_B4B-XH-A_1x04_P2.50mm_Vertical
- removed J12: Limit_Min, Connector_JST:JST_XH_B2B-XH-A_1x02_P2.50mm_Vertical
- removed J13: Limit_Max, Connector_JST:JST_XH_B2B-XH-A_1x02_P2.50mm_Vertical
- removed J14: Limit_Z_Home, Connector_JST:JST_XH_B2B-XH-A_1x02_P2.50mm_Vertical
- removed J2: USB_PROG, Connector_USB:USB_C_Receptacle_GCT_USB4085
- removed J4: Motor_Pan, Connector_JST:JST_XH_B4B-XH-A_1x04_P2.50mm_Vertical
- removed J5: Motor_Tilt, Connector_JST:JST_XH_B4B-XH-A_1x04_P2.50mm_Vertical
- removed J6: Motor_Z, Connector_JST:JST_XH_B4B-XH-A_1x04_P2.50mm_Vertical
- removed J7: AS5600_Pan, Connector_JST:JST_XH_B4B-XH-A_1x04_P2.50mm_Vertical
- removed J8: AS5600_Tilt, Connector_JST:JST_XH_B4B-XH-A_1x04_P2.50mm_Vertical
- removed J9: OLED, Connector_JST:JST_XH_B4B-XH-A_1x04_P2.50mm_Vertical
- removed R1, R2: 10k, Resistor_SMD:R_0603_1608Metric
- removed R12, R13, R6: 0.11, Resistor_SMD:R_0603_1608Metric
- removed R14, R15, R16, R17, R18, R19, R20, R21: 4.7k, Resistor_SMD:R_0603_1608Metric
- removed R3, R4: 5.1k, Resistor_SMD:R_0603_1608Metric
- removed R5: 1k, Resistor_SMD:R_0603_1608Metric
- removed SW1: BOOT, Button_Switch_THT:SW_PUSH_6mm
- removed SW2: RESET, Button_Switch_THT:SW_PUSH_6mm
- removed U3: ESP32-S3-WROOM-1-N16R8, RF_Module:ESP32-S3-WROOM-1
- removed U5, U6, U7: TMC2209-LA, Package_DFN_QFN:VQFN-28-1EP_5x5mm_P0.5mm_EP3.7x3.7mm_ThermalVias
- removed U8: TCA9548APWR, Package_SO:TSSOP-24_4.4x7.8mm_P0.65mm
- added C56: 100nF, Capacitor_SMD:C_0603_1608Metric, F.Cu at (199.4, 81.2)
- added C57: 100nF, Capacitor_SMD:C_0603_1608Metric, F.Cu at (242.1, 65.7)
- added C58: 100nF, Capacitor_SMD:C_0603_1608Metric, F.Cu at (242.1, 106.3)
- added C59: 100uF_35V, Capacitor_THT:CP_Radial_D8.0mm_P3.50mm, F.Cu at (234.4, 66.2)
- added C60: 100uF_35V, Capacitor_THT:CP_Radial_D8.0mm_P3.50mm, F.Cu at (234.4, 106.8)
- added C61: 100nF, Capacitor_SMD:C_0603_1608Metric, F.Cu at (250.3, 73.2)
- added C62: 100nF, Capacitor_SMD:C_0603_1608Metric, F.Cu at (250.3, 113.8)
- added C63: 100nF, Capacitor_SMD:C_0603_1608Metric, F.Cu at (241.3, 71.3)
- added C64: 100nF, Capacitor_SMD:C_0603_1608Metric, F.Cu at (241.3, 111.9)
- added C65: 4.7uF, Capacitor_SMD:C_0603_1608Metric, F.Cu at (244.6, 75.1)
- added C66: 4.7uF, Capacitor_SMD:C_0603_1608Metric, F.Cu at (244.6, 115.7)
- added C67: 22nF, Capacitor_SMD:C_0603_1608Metric, F.Cu at (239.5, 68.6)
- added C68: 22nF, Capacitor_SMD:C_0603_1608Metric, F.Cu at (239.5, 109.2)
- added C69: 100nF, Capacitor_SMD:C_0603_1608Metric, F.Cu at (250.3, 93.5)
- added C70: 100nF, Capacitor_THT:CP_Radial_D8.0mm_P3.50mm, F.Cu at (234.4, 86.5)
- added C71: 100nF, Capacitor_SMD:C_0603_1608Metric, F.Cu at (242.1, 126.6)
- added C72: 100uF_35V, Capacitor_SMD:C_0603_1608Metric, F.Cu at (242.1, 86.0)
- added C73: 100uF_35V, Capacitor_THT:CP_Radial_D8.0mm_P3.50mm, F.Cu at (234.4, 127.1)
- added C74: 100nF, Capacitor_SMD:C_0603_1608Metric, F.Cu at (250.3, 134.1)
- added C75: 100nF, Capacitor_SMD:C_0603_1608Metric, F.Cu at (241.3, 91.6)
- added C76: 100nF, Capacitor_SMD:C_0603_1608Metric, F.Cu at (241.3, 132.2)
- added C77: 4.7uF, Capacitor_SMD:C_0603_1608Metric, F.Cu at (244.6, 95.4)
- added C78: 22nF, Capacitor_SMD:C_0603_1608Metric, F.Cu at (239.5, 88.9)
- added C79: 22nF, Capacitor_SMD:C_0603_1608Metric, F.Cu at (239.5, 129.5)
- added C80: 4.7uF, Capacitor_SMD:C_0603_1608Metric, F.Cu at (244.6, 136.0)
- added D3: SS34, Diode_SMD:D_SMC, F.Cu at (123.2, 179.1)
- added J19: AS5600_Pan, Connector_JST:JST_XH_B4B-XH-A_1x04_P2.50mm_Vertical, F.Cu at (177.0, 83.3)
- added J20: AS5600_Tilt, Connector_JST:JST_XH_B4B-XH-A_1x04_P2.50mm_Vertical, F.Cu at (177.0, 91.1)
- added J21: OLED, Connector_JST:JST_XH_B4B-XH-A_1x04_P2.50mm_Vertical, F.Cu at (177.0, 98.9)
- added J22: Enc_Jog, Connector_JST:JST_XH_B4B-XH-A_1x04_P2.50mm_Vertical, F.Cu at (177.0, 106.7)
- added J23: Enc_Angle, Connector_JST:JST_XH_B4B-XH-A_1x04_P2.50mm_Vertical, F.Cu at (177.0, 114.5)
- added J24: Limit_Min, Connector_JST:JST_XH_B2B-XH-A_1x02_P2.50mm_Vertical, F.Cu at (191.4, 83.3)
- added J25: Limit_Max, Connector_JST:JST_XH_B2B-XH-A_1x02_P2.50mm_Vertical, F.Cu at (191.4, 91.1)
- added J26: Limit_Z_Home, Connector_JST:JST_XH_B2B-XH-A_1x02_P2.50mm_Vertical, F.Cu at (191.4, 98.9)
- added J27: Motor_Slide, Connector_JST:JST_XH_B4B-XH-A_1x04_P2.50mm_Vertical, F.Cu at (257.3, 71.8)
- added J28: Motor_Tilt, Connector_JST:JST_XH_B4B-XH-A_1x04_P2.50mm_Vertical, F.Cu at (257.3, 112.5)
- added J29: Motor_Pan, Connector_JST:JST_XH_B4B-XH-A_1x04_P2.50mm_Vertical, F.Cu at (257.3, 92.1)
- added J30: Motor_Z, Connector_JST:JST_XH_B4B-XH-A_1x04_P2.50mm_Vertical, F.Cu at (257.3, 132.8)
- added R30: 4.7k, Resistor_SMD:R_0603_1608Metric, F.Cu at (199.4, 83.7)
- added R31: 4.7k, Resistor_SMD:R_0603_1608Metric, F.Cu at (199.4, 86.2)
- added R32: 4.7k, Resistor_SMD:R_0603_1608Metric, F.Cu at (199.4, 88.7)
- added R33: 4.7k, Resistor_SMD:R_0603_1608Metric, F.Cu at (199.4, 91.2)
- added R34: 4.7k, Resistor_SMD:R_0603_1608Metric, F.Cu at (199.4, 93.7)
- added R35: 4.7k, Resistor_SMD:R_0603_1608Metric, F.Cu at (199.4, 96.2)
- added R36: 4.7k, Resistor_SMD:R_0603_1608Metric, F.Cu at (199.4, 98.7)
- added R37: 4.7k, Resistor_SMD:R_0603_1608Metric, F.Cu at (199.4, 101.2)
- added R38: 0.11, Resistor_SMD:R_0603_1608Metric, F.Cu at (244.6, 63.0)
- added R39: 0.11, Resistor_SMD:R_0603_1608Metric, F.Cu at (244.6, 103.6)
- added R40: 0.11, Resistor_SMD:R_0603_1608Metric, F.Cu at (247.8, 63.0)
- added R41: 0.11, Resistor_SMD:R_0603_1608Metric, F.Cu at (247.8, 103.6)
- added R42: 0.11, Resistor_SMD:R_0603_1608Metric, F.Cu at (247.8, 83.3)
- added R43: 0.11, Resistor_SMD:R_0603_1608Metric, F.Cu at (244.6, 124.0)
- added R44: 0.11, Resistor_SMD:R_0603_1608Metric, F.Cu at (244.6, 83.3)
- added R45: 0.11, Resistor_SMD:R_0603_1608Metric, F.Cu at (247.8, 124.0)
- added SW3: RESET, Button_Switch_THT:SW_PUSH_6mm, F.Cu at (51.6, 99.1)
- added SW4: BOOT, Button_Switch_THT:SW_PUSH_6mm, F.Cu at (79.2, 111.7)
- added U13: TCA9548APWR, Package_SO:TSSOP-24_4.4x7.8mm_P0.65mm, F.Cu at (192.7, 108.0)
- added U14: TMC2209-LA, Package_DFN_QFN:VQFN-28-1EP_5x5mm_P0.5mm_EP3.7x3.7mm_ThermalVias, F.Cu at (246.4, 69.2)
- added U15: TMC2209-LA, Package_DFN_QFN:VQFN-28-1EP_5x5mm_P0.5mm_EP3.7x3.7mm_ThermalVias, F.Cu at (246.4, 109.9)
- added U16: TMC2209-LA, Package_DFN_QFN:VQFN-28-1EP_5x5mm_P0.5mm_EP3.7x3.7mm_ThermalVias, F.Cu at (246.4, 89.5)
- added U17: TMC2209-LA, Package_DFN_QFN:VQFN-28-1EP_5x5mm_P0.5mm_EP3.7x3.7mm_ThermalVias, F.Cu at (246.4, 130.2)
- C11: value 22nF -> 22uF
- C12: value 100nF -> 1uF
- C13: value 4.7uF -> 100nF
- C14: value 100nF -> 10uF; footprint Capacitor_SMD:C_0603_1608Metric -> Capacitor_SMD:C_0805_2012Metric
- C15: value 100uF_35V -> 100nF; footprint Capacitor_THT:CP_Radial_D8.0mm_P3.50mm -> Capacitor_SMD:C_0603_1608Metric
- C16: value 22nF -> 100nF
- C5: value 22uF -> 0.1uF
- J3: value Motor_Slide -> USB_PROG; footprint Connector_JST:JST_XH_B4B-XH-A_1x04_P2.50mm_Vertical -> Connector_USB:USB_C_Receptacle_GCT_USB4085
- R10: value 0.11 -> 1k
- R11, R9: value 0.11 -> 10k
- R7, R8: value 0.11 -> 5.1k
- U4: value TMC2209-LA -> ESP32-S3-WROOM-1-N16R8; footprint Package_DFN_QFN:VQFN-28-1EP_5x5mm_P0.5mm_EP3.7x3.7mm_ThermalVias -> RF_Module:ESP32-S3-WROOM-1
- moved C12 186.8 mm to (224.5, 19.8)
- moved C13 186.8 mm to (224.5, 22.3)
- moved R7 185.9 mm to (242.2, 19.8)
- moved C15 184.1 mm to (224.5, 24.8)
- moved R10 167.6 mm to (224.5, 32.4)
- moved R11 167.6 mm to (224.5, 34.9)
- moved R9 152.2 mm to (51.2, 103.5), turned to 0 degrees
- moved J3 146.0 mm to (66.9, 175.0), turned to 0 degrees
- moved C14 131.9 mm to (186.3, 62.3)
- moved C11 110.0 mm to (123.2, 167.6), turned to 90 degrees
- moved U4 87.6 mm to (67.3, 99.1)
- moved F1 85.5 mm to (81.3, 181.4), turned to 90 degrees
- moved J1 84.6 mm to (88.2, 179.1)
- moved U2 58.0 mm to (129.5, 168.9), turned to 0 degrees
- moved R8 52.5 mm to (242.2, 22.3), turned to 0 degrees
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Connections:
- net /+24V_RAW renamed /power/+24V_RAW
- C11 pad 1: CP_Slide -> +3V3
- C11 pad 2: CP_Slide_B -> GND
- C12 pad 1: VCP_Slide -> EN_ESP
- C12 pad 2: Net-(C12-Pad2) -> GND
- C13 pad 1: 5VOUT_Slide -> +3V3
- C13 pad 2: unconnected-(C13-Pad2) -> GND
- C14 pad 1: Net-(C12-Pad2) -> +3V3
- C15 pad 1: Net-(C12-Pad2) -> +3V3
- C16 pad 1: CP_Pan -> +3V3
- C16 pad 2: CP_Pan_B -> GND
- D1 pad 1: unconnected-(D1-K-Pad1) -> /power/SW_NODE
- L1 pad 2: GND -> /power/SW_NODE
- R10 pad 1: RSA_Tilt -> GPIO47
- R10 pad 2: GND -> TMC_UART
- R11 pad 1: RSB_Tilt -> GPIO0
- R11 pad 2: GND -> +3V3
- R7 pad 1: RSB_Slide -> USBCC1
- R8 pad 1: RSA_Pan -> USBCC2
- R9 pad 1: RSB_Pan -> EN_ESP
- R9 pad 2: GND -> +3V3
- U1 pad 2: GND -> /power/SW_NODE
- U4 pad 1: MOTOR_Slide_B2 -> GND
- U4 pad 10: GND -> GPIO17
- U4 pad 11: unconnected-(U4-DIAG-Pad11) -> GPIO18
- U4 pad 12: unconnected-(U4-INDEX-Pad12) -> GPIO8
- U4 pad 13: GND -> GPIO19
- U4 pad 14: TMC_UART -> GPIO20
- U4 pad 15: +3V3 -> unconnected-(U4-IO3-Pad15)
- U4 pad 16: GPIO4 -> unconnected-(U4-IO46-Pad16)
- U4 pad 17: unconnected-(U4-VREF-Pad17) -> GPIO9
- U4 pad 18: GND -> GPIO10
- U4 pad 19: GPIO5 -> GPIO11
- U4 pad 2: GPIO10 -> +3V3
- U4 pad 20: unconnected-(U4-STDBY-Pad20) -> GPIO12
- U4 pad 21: MOTOR_Slide_A2 -> GPIO13
- U4 pad 22: Net-(C12-Pad2) -> GPIO14
- U4 pad 23: RSA_Slide -> GPIO21
- U4 pad 24: MOTOR_Slide_A1 -> GPIO47
- U4 pad 26: MOTOR_Slide_B1 -> unconnected-(U4-IO45-Pad26)
- U4 pad 27: RSB_Slide -> GPIO0
- U4 pad 28: Net-(C12-Pad2) -> unconnected-(U4-IO35-Pad28)
- U4 pad 29: GND -> unconnected-(U4-IO36-Pad29)
- U4 pad 3: GND -> EN_ESP
- U4 pad 4: CP_Slide_B -> GPIO4
- U4 pad 5: CP_Slide -> GPIO5
- U4 pad 6: VCP_Slide -> GPIO6
- U4 pad 7: GND -> GPIO7
- U4 pad 8: 5VOUT_Slide -> GPIO15
- U4 pad 9: GND -> GPIO16
Routing:
- net +24V: track 21.3 -> 42.7 mm
- net +5V: track 18.4 -> 0.00 mm
- net /stepper drivers/M3_B2: track 0.00 -> 17.9 mm, vias 0 -> 1
- net /stepper drivers/M2_B2: track 0.00 -> 17.9 mm, vias 0 -> 1
- net /stepper drivers/M1_B2: track 0.00 -> 17.9 mm, vias 0 -> 1
- net /stepper drivers/M0_B2: track 0.00 -> 17.9 mm, vias 0 -> 1
- net /stepper drivers/M3_A1: track 0.00 -> 14.4 mm, vias 0 -> 1
- net /stepper drivers/M1_A1: track 0.00 -> 14.4 mm, vias 0 -> 1
- net /stepper drivers/M2_A1: track 0.00 -> 14.4 mm, vias 0 -> 1
- net /stepper drivers/M0_A1: track 0.00 -> 14.4 mm, vias 0 -> 1
- net /stepper drivers/M3_B1: track 0.00 -> 13.7 mm, vias 0 -> 1
- net /stepper drivers/M1_B1: track 0.00 -> 13.7 mm, vias 0 -> 1
- net /stepper drivers/M2_B1: track 0.00 -> 13.7 mm, vias 0 -> 1
- net /stepper drivers/M0_B1: track 0.00 -> 13.7 mm, vias 0 -> 1
- net MOTOR_Slide_A2: track 12.3 -> 0.00 mm
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- removed copper zone on In2.Cu, net +3V3
- removed copper zone on B.Cu, net GND
- removed copper zone on F.Cu, net GND
- removed copper zone on In1.Cu, net GND
Other:
- board outline removed
