File: integrated/schematic/pantiltslide_integrated.kicad_sch (KiCad schematic)
At the start: 82 parts, among them J1 24V_In, J10 Limit_Min, J11 Limit_Max, J12 Limit_Z_Home, J2 USB_PROG, J3 Motor_Slide, J4 Motor_Pan, J5 Motor_Tilt, J6 Motor_Z, J7 OLED, J8 Enc_Jog, J9 Enc_Angle, SW1 BOOT, SW2 RESET, U1 LM2596S-5, U10 AS5600-ASOT, U2 AMS1117-3.3, U3 ESP32-S3-WROOM-1-N16R8, U4 TMC2209-LA, U5 TMC2209-LA, U6 TMC2209-LA, U7 TMC2209-LA, U8 TCA9548APWR, U9 AS5600-ASOT

Commit message: upfsd
Parts:
- removed C32, C33: 100nF, Capacitor_SMD:C_0603_1608Metric, symbol Device:C
- removed J10: Limit_Min, TerminalBlock:TerminalBlock_Altech_AK300-2_P5.00mm, symbol Connector:Screw_Terminal_01x02
- removed J11: Limit_Max, TerminalBlock:TerminalBlock_Altech_AK300-2_P5.00mm, symbol Connector:Screw_Terminal_01x02
- removed U10, U9: AS5600-ASOT, Package_SO:SOIC-8_3.9x4.9mm_P1.27mm, symbol New_Library:AS5600
- added J10: Enc_Jog, Connector_PinHeader_2.54mm:PinHeader_1x04_P2.54mm_Vertical, symbol Connector:Conn_01x04_Pin
- added J11: Enc_Angle, Connector_PinHeader_2.54mm:PinHeader_1x04_P2.54mm_Vertical, symbol Connector:Conn_01x04_Pin
- added J13: Limit_Max, TerminalBlock:TerminalBlock_Altech_AK300-2_P5.00mm, symbol Connector:Screw_Terminal_01x02
- added J14: Limit_Z_Home, TerminalBlock:TerminalBlock_Altech_AK300-2_P5.00mm, symbol Connector:Screw_Terminal_01x02
- J12: value Limit_Z_Home -> Limit_Min
- J7: value OLED -> AS5600_Pan
- J8: value Enc_Jog -> AS5600_Tilt
- J9: value Enc_Angle -> OLED
Connections:
- net +24V: now also C1.1, C12.2, C14.1, C15.1, C17.2, C19.1, C2.1, C20.1, C22.2, C24.1, C25.1, C27.2, C29.1, C30.1, U1.1 (VIN), U4.22 (VS), U4.28 (VS), U5.22 (VS), U5.28 (VS), U6.22 (VS), U6.28 (VS), U7.22 (VS), U7.28 (VS); no longer C1.2, C12.1, C14.2, C15.2, C17.1, C19.2, C2.2, C20.2, C22.1, C24.2, C25.2, C27.1, C29.2, C30.2, U1.5 (~{ON}/OFF)
- net +3V3: now also J7.1 (Pin_1), J8.1 (Pin_1), J9.1 (Pin_1), R1.2, R14.2, R15.2, R16.2, R17.2, R18.2, R19.2, R2.2, R20.2, R21.2, U3.2 (3V3), U4.15 (VCC_IO), U5.15 (VCC_IO), U6.15 (VCC_IO), U7.15 (VCC_IO), U8.24 (VCC), U8.3 (~{RESET}); no longer C1.1, C10.2, C13.1, C14.1, C15.1, C18.1, C19.1, C2.1, C20.1, C23.1, C24.1, C25.1, C28.1, C29.1, C3.1, C30.1, C31.2, C4.1, C5.2, C6.1, C7.2, C8.2, C9.2, D1.2 (A), J7.2 (Pin_2), J7.3 (Pin_3), R1.1, R10.1, R11.1, R12.1, R13.1, R14.1, R15.1, R16.1, R17.1, R18.1, R19.1, R2.1, R20.1, R21.1, R3.1, R4.1, R6.1, R7.1, R8.1, R9.1, SW1.2, SW2.2, U1.1 (VIN), U3.20 (IO12), U3.21 (IO13), U3.23 (IO21), U3.24 (IO47), U4.10 (MS2/AD1), U4.22 (VS), U4.28 (VS), U4.7 (SPREAD), U4.9 (MS1/AD0), U5.10 (MS2/AD1), U5.22 (VS), U5.28 (VS), U5.7 (SPREAD), U6.22 (VS), U6.28 (VS), U6.7 (SPREAD), U6.9 (MS1/AD0), U7.22 (VS), U7.28 (VS), U7.7 (SPREAD), U8.12 (GND)
- net +5V: now also C3.1, C4.1, L1.2, U1.4 (FB); no longer C3.2, C4.2, L1.1, U1.2 (OUT)
- net 5VOUT_Pan: now also C18.1, U5.8 (5VOUT); no longer C18.2
- net 5VOUT_Slide: now also C13.1, U4.8 (5VOUT); no longer C13.2
- net 5VOUT_Tilt: now also C23.1, U6.8 (5VOUT); no longer C23.2
- net 5VOUT_Z: now also C28.1, U7.8 (5VOUT); no longer C28.2
- net CP_Pan: now also C16.1, U5.5 (CPI); no longer C16.2
- net CP_Pan_B: now also C16.2, U5.4 (CPO); no longer C16.1, U5.1 (OB2)
- net CP_Slide: now also C11.1, U4.5 (CPI); no longer C11.2
- net CP_Slide_B: now also C11.2, U4.4 (CPO); no longer C11.1, U4.1 (OB2)
- net CP_Tilt: now also C21.1, U6.5 (CPI); no longer C21.2
- net CP_Tilt_B: now also C21.2, U6.4 (CPO); no longer C21.1, U6.1 (OB2)
- net CP_Z: now also C26.1, U7.5 (CPI); no longer C26.2
- net CP_Z_B: now also C26.2, U7.4 (CPO); no longer C26.1, U7.1 (OB2)
- net EN_ESP: now also C6.1, R1.1, U3.3 (EN); no longer C6.2, R1.2, U3.19 (IO11)
- net GPIO0: now also R2.1, U3.27 (IO0); no longer R2.2, U3.37 (TXD0)
- net GPIO1: now also U3.39 (IO1), U7.16 (STEP); no longer U3.25 (IO48)
- net GPIO10: now also U3.18 (IO10), U4.2 (~{EN}), U5.2 (~{EN}), U6.2 (~{EN}), U7.2 (~{EN}); no longer U3.4 (IO4), U4.14 (~{PD}/UART), U5.14 (~{PD}/UART), U6.14 (~{PD}/UART), U7.14 (~{PD}/UART)
- net GPIO11: now also R14.1, U3.19 (IO11), U8.23 (SDA); no longer R14.2, U3.3 (EN)
- net GPIO12: now also R15.1, U3.20 (IO12), U8.22 (SCL); no longer R15.2, U3.2 (3V3)
- net GPIO13: now also J9.3 (Pin_3), R20.1, U3.21 (IO13); no longer J7.1 (Pin_1), R20.2, U3.1 (GND)
- net GPIO14: now also J9.4 (Pin_4), R21.1, U3.22 (IO14); no longer R21.2
- net GPIO15: now also U3.8 (IO15), J10.1 (Pin_1); no longer J8.3 (Pin_3), U3.14 (IO20)
- net GPIO16: now also U3.9 (IO16), J10.2 (Pin_2); no longer J8.2 (Pin_2), U3.13 (IO19)
- net GPIO17: now also U3.10 (IO17), J10.3 (Pin_3); no longer J8.1 (Pin_1), U3.12 (IO8)
- net GPIO18: now also J11.1 (Pin_1); no longer J9.3 (Pin_3)
- net GPIO19: now also J2.A7 (D-), J2.B7 (D-), U3.13 (IO19); no longer J2.A6 (D+), U3.9 (IO16)
- net GPIO2: now also U3.38 (IO2), U7.19 (DIR); no longer U3.26 (IO45), U7.12 (INDEX)
- net GPIO20: now also J2.A6 (D+), J2.B6 (D+), U3.14 (IO20); no longer J2.A7 (D-), U3.8 (IO15)
- net GPIO21: now also U3.23 (IO21), J11.2 (Pin_2); no longer J9.2 (Pin_2), U3.41 (GND)
- net GPIO38: now also U3.31 (IO38), J11.3 (Pin_3); no longer J9.1 (Pin_1), U3.33 (IO40)
- net GPIO39: now also J12.1 (Pin_1)
- net GPIO4: now also U3.4 (IO4), U4.16 (STEP); no longer U3.18 (IO10)
- net GPIO40: now also U3.33 (IO40), J13.1 (Pin_1); no longer U3.31 (IO38)
- net GPIO42: now also U3.35 (IO42), J14.1 (Pin_1); no longer J12.1 (Pin_1), U3.29 (IO36)
- net GPIO47: now also R5.1, U3.24 (IO47); no longer R5.2, U3.40 (GND)
- net GPIO5: now also U3.5 (IO5), U4.19 (DIR); no longer U3.17 (IO9), U4.12 (INDEX)
- net GPIO6: now also U3.6 (IO6), U5.16 (STEP); no longer U3.16 (IO46)
- net GPIO7: now also U3.7 (IO7), U5.19 (DIR); no longer U3.15 (IO3), U5.12 (INDEX)
- net GPIO8: now also U3.12 (IO8), U6.16 (STEP); no longer U3.10 (IO17)
- net GPIO9: now also U3.17 (IO9), U6.19 (DIR); no longer U3.5 (IO5), U6.12 (INDEX)
- net I2C_PAN_SCL: now also J7.4 (Pin_4), R17.1, U8.5 (SC0); no longer R17.2, U8.20 (SC7)
- net I2C_PAN_SDA: now also J7.3 (Pin_3), R16.1, U8.4 (SD0); no longer R16.2, U8.17 (SD6)
- net I2C_TILT_SCL: now also J8.4 (Pin_4), R19.1, U8.7 (SC1); no longer R19.2, U8.18 (SC6)
- net I2C_TILT_SDA: now also J8.3 (Pin_3), R18.1, U8.6 (SD1); no longer R18.2, U8.15 (SD5)
- net MOTOR_Pan_A1: now also J4.1 (Pin_1); no longer J4.3 (Pin_3)
- net MOTOR_Pan_A2: now also U5.21 (OA2)
- net MOTOR_Pan_B1: now also J4.3 (Pin_3), U5.26 (OB1); no longer J4.1 (Pin_1)
- net MOTOR_Pan_B2: now also J4.4 (Pin_4), U5.1 (OB2); no longer U5.4 (CPO)
- net MOTOR_Slide_A1: now also J3.1 (Pin_1); no longer J3.3 (Pin_3)
- net MOTOR_Slide_A2: now also U4.21 (OA2)
- net MOTOR_Slide_B1: now also J3.3 (Pin_3), U4.26 (OB1); no longer J3.1 (Pin_1)
- net MOTOR_Slide_B2: now also J3.4 (Pin_4), U4.1 (OB2); no longer U4.4 (CPO)
- net MOTOR_Tilt_A1: now also J5.1 (Pin_1); no longer J5.3 (Pin_3)
- net MOTOR_Tilt_A2: now also U6.21 (OA2)
- net MOTOR_Tilt_B1: now also J5.3 (Pin_3), U6.26 (OB1); no longer J5.1 (Pin_1)
- net MOTOR_Tilt_B2: now also J5.4 (Pin_4), U6.1 (OB2); no longer U6.4 (CPO)
- net MOTOR_Z_A1: now also J6.1 (Pin_1); no longer J6.3 (Pin_3)
- net MOTOR_Z_A2: now also U7.21 (OA2)
- net MOTOR_Z_B1: now also J6.3 (Pin_3), U7.26 (OB1); no longer J6.1 (Pin_1)
- net MOTOR_Z_B2: now also J6.4 (Pin_4), U7.1 (OB2); no longer U7.4 (CPO)
- net RSA_Pan: now also R8.1, U5.23 (BRA); no longer R8.2, U5.17 (VREF)
- net RSA_Slide: now also R6.1, U4.23 (BRA); no longer R6.2, U4.17 (VREF)
- net RSA_Tilt: now also R10.1, U6.23 (BRA); no longer R10.2, U6.17 (VREF)
- net RSA_Z: now also R12.1, U7.23 (BRA); no longer R12.2, U7.17 (VREF)
- net RSB_Pan: now also R9.1, U5.27 (BRB); no longer R9.2
- net RSB_Slide: now also R7.1, U4.27 (BRB); no longer R7.2
- net RSB_Tilt: now also R11.1, U6.27 (BRB); no longer R11.2
- net RSB_Z: now also R13.1, U7.27 (BRB); no longer R13.2
- net SW_NODE: now also L1.1, U1.2 (OUT); no longer L1.2, U1.4 (FB)
- net TMC_UART: now also R5.2, U3.34 (IO41), U4.14 (~{PD}/UART), U5.14 (~{PD}/UART), U6.14 (~{PD}/UART), U7.14 (~{PD}/UART); no longer R5.1, U3.30 (IO37), U4.2 (~{EN}), U5.2 (~{EN}), U6.2 (~{EN}), U7.2 (~{EN})
- net USBCC1: now also J2.A5 (CC1), R3.1; no longer R3.2
- net USBCC2: now also J2.B5 (CC2), R4.1; no longer R4.2
- net USB_VBUS: now also J2.A4 (VBUS), J2.A9 (VBUS), J2.B4 (VBUS), J2.B9 (VBUS)
- net VCP_Pan: now also C17.1, U5.6 (VCP); no longer C17.2
- net VCP_Slide: now also C12.1, U4.6 (VCP); no longer C12.2
- net VCP_Tilt: now also C22.1, U6.6 (VCP); no longer C22.2
- net VCP_Z: now also C27.1, U7.6 (VCP); no longer C27.2
- net GND: now reaches J12.2 (Pin_2)
- net GND: now also C1.2, C10.2, C13.2, C14.2, C15.2, C18.2, C19.2, C2.2, C20.2, C23.2, C24.2, C25.2, C28.2, C29.2, C3.2, C30.2, C31.2, C4.2, C5.2, C6.2, C7.2, C8.2, C9.2, D1.2 (A), J1.2 (Pin_2), J2.A1 (GND), J2.A12 (GND), J2.B1 (GND), J2.B12 (GND), J2.S1 (SHIELD), J7.2 (Pin_2), J8.2 (Pin_2), J9.2 (Pin_2), R10.2, R11.2, R12.2, R13.2, R3.2, R4.2, R6.2, R7.2, R8.2, R9.2, SW1.2, SW2.2, U1.3 (GND), U1.5 (~{ON}/OFF), U2.1 (GND), U3.1 (GND), U3.40 (GND), U3.41 (GND), U4.10 (MS2/AD1), U4.13 (CLK), U4.18 (GND), U4.29 (GND), U4.3 (GND), U4.7 (SPREAD), U4.9 (MS1/AD0), U5.10 (MS2/AD1), U5.13 (CLK), U5.18 (GND), U5.29 (GND), U5.3 (GND), U5.7 (SPREAD), U6.13 (CLK), U6.18 (GND), U6.29 (GND), U6.3 (GND), U6.7 (SPREAD), U6.9 (MS1/AD0), U7.13 (CLK), U7.18 (GND), U7.29 (GND), U7.3 (GND), U7.7 (SPREAD), U8.1 (A0), U8.12 (GND), U8.2 (A1), U8.21 (A2), J10.4 (Pin_4), J11.4 (Pin_4), J13.2 (Pin_2), J14.2 (Pin_2)
- no-connect marks 55 -> 41

Commit message: updates
Parts:
- removed J12: Limit_Min, TerminalBlock:TerminalBlock_Altech_AK300-2_P5.00mm, symbol Connector:Screw_Terminal_01x02
- removed J13: Limit_Max, TerminalBlock:TerminalBlock_Altech_AK300-2_P5.00mm, symbol Connector:Screw_Terminal_01x02
- removed J14: Limit_Z_Home, TerminalBlock:TerminalBlock_Altech_AK300-2_P5.00mm, symbol Connector:Screw_Terminal_01x02
- added J12: Limit_Min, Connector_JST:JST_XH_B2B-XH-A_1x02_P2.50mm_Vertical, symbol Connector:Conn_01x02_Pin
- added J13: Limit_Max, Connector_JST:JST_XH_B2B-XH-A_1x02_P2.50mm_Vertical, symbol Connector:Conn_01x02_Pin
- added J14: Limit_Z_Home, Connector_JST:JST_XH_B2B-XH-A_1x02_P2.50mm_Vertical, symbol Connector:Conn_01x02_Pin
- J10, J11, J3, J4, J5, J6, J7, J8, J9: footprint Connector_PinHeader_2.54mm:PinHeader_1x04_P2.54mm_Vertical -> Connector_JST:JST_XH_B4B-XH-A_1x04_P2.50mm_Vertical
Connections:
- net GND: now also J12.2 (Pin_2), J13.2 (Pin_2), J14.2 (Pin_2)
- net GPIO39: now also J12.1 (Pin_1)
- net GPIO40: now also J13.1 (Pin_1)
- net GPIO42: now also J14.1 (Pin_1)
Other:
- note added: "I2C MUX + OFF-BOARD I/O CONNECTORS"
- note added: "MCU ESP32-S3-WROOM-1 + USB-C"
- note added: "POWER 24V IN / 5V BUCK / 3V3 LDO"
- note added: "STEPPER DRIVERS 4x TMC2209"

Commit message: latest version
Parts:
- removed C10: 10uF, Capacitor_THT:CP_Radial_D8.0mm_P3.50mm, symbol Device:C_Polarized
- added C10: 10uF, Capacitor_SMD:C_0805_2012Metric, symbol Device:C
- C1, C2: Decouples (none) -> U1 +24V
- C12, C14, C15: Decouples (none) -> U4 +24V
- C13: Decouples (none) -> U4 5VOUT_Slide
- C17, C19, C20: Decouples (none) -> U5 +24V
- C18: Decouples (none) -> U5 5VOUT_Pan
- C22, C24, C25: Decouples (none) -> U6 +24V
- C23: Decouples (none) -> U6 5VOUT_Tilt
- C27, C29, C30: Decouples (none) -> U7 +24V
- C28: Decouples (none) -> U7 5VOUT_Z
- C3: Decouples (none) -> U1 +5V
- C31: Decouples (none) -> U8 +3V3
- C4: Decouples (none) -> U2 +5V
- C5: Decouples (none) -> U2 +3V3
- C7, C8, C9: Decouples (none) -> U3 +3V3
Connections:
- net +3V3 is gone; now on net +24V: C31.1, C5.1, C7.1, C8.1, C9.1, J7.1 (Pin_1), J8.1 (Pin_1), J9.1 (Pin_1), R1.2, R14.2, R15.2, R16.2, R17.2, R18.2, R19.2, R2.2, R20.2, R21.2, U2.2 (VO), U3.2 (3V3), U4.15 (VCC_IO), U5.15 (VCC_IO), U5.9 (MS1/AD0), U6.10 (MS2/AD1), U6.15 (VCC_IO), U7.10 (MS2/AD1), U7.15 (VCC_IO), U7.9 (MS1/AD0), U8.24 (VCC), U8.3 (~{RESET})
- net 5VOUT_Pan is gone; now on net +24V: C18.1, U5.8 (5VOUT)
- net 5VOUT_Slide is gone; now on net +24V: C13.1, U4.8 (5VOUT)
- net 5VOUT_Tilt is gone; now on net +24V: C23.1, U6.8 (5VOUT)
- net 5VOUT_Z is gone; now on net +24V: C28.1, U7.8 (5VOUT)
- net GND is gone; now on net +24V: C1.2, C13.2, C14.2, C15.2, C18.2, C19.2, C2.2, C20.2, C23.2, C24.2, C25.2, C28.2, C29.2, C3.2, C30.2, C31.2, C4.2, C5.2, C6.2, C7.2, C8.2, C9.2, D1.2 (A), J1.2 (Pin_2), J10.4 (Pin_4), J11.4 (Pin_4), J12.2 (Pin_2), J13.2 (Pin_2), J14.2 (Pin_2), J2.A1 (GND), J2.A12 (GND), J2.B1 (GND), J2.B12 (GND), J2.S1 (SHIELD), J7.2 (Pin_2), J8.2 (Pin_2), J9.2 (Pin_2), R10.2, R11.2, R12.2, R13.2, R3.2, R4.2, R6.2, R7.2, R8.2, R9.2, SW1.2, SW2.2, U1.3 (GND), U1.5 (~{ON}/OFF), U2.1 (GND), U3.1 (GND), U3.40 (GND), U3.41 (GND), U4.10 (MS2/AD1), U4.13 (CLK), U4.18 (GND), U4.29 (GND), U4.3 (GND), U4.7 (SPREAD), U4.9 (MS1/AD0), U5.10 (MS2/AD1), U5.13 (CLK), U5.18 (GND), U5.29 (GND), U5.3 (GND), U5.7 (SPREAD), U6.13 (CLK), U6.18 (GND), U6.29 (GND), U6.3 (GND), U6.7 (SPREAD), U6.9 (MS1/AD0), U7.13 (CLK), U7.18 (GND), U7.29 (GND), U7.3 (GND), U7.7 (SPREAD), U8.1 (A0), U8.12 (GND), U8.2 (A1), U8.21 (A2)
- net SW_NODE is gone; now on net +24V: D1.1 (K), L1.1, U1.2 (OUT)
- net +24V: now also C3.1, C4.1, D2.1 (K), L1.2, U1.4 (FB), U2.3 (VI), C10.1, C10.2; no longer F1.1, J1.1 (Pin_1)
- net USB_VBUS: now also D2.2 (A); no longer D2.1 (K)
- removed net +5V: C3.1, C4.1, D2.2 (A), L1.2, U1.4 (FB), U2.3 (VI)
- new net +24V_RAW: F1.1, J1.1 (Pin_1)

Commit message: switching tmc2209s to new schmatic file
Parts:
- J1: footprint TerminalBlock:TerminalBlock_Altech_AK300-2_P5.00mm -> TerminalBlock:TerminalBlock_MaiXu_MX126-5.0-02P_1x02_P5.00mm
Connections:
- net +24V: no longer C1.2, C10.1, C10.2, C12.2, C13.1, C13.2, C14.1, C14.2, C15.1, C15.2, C18.1, C18.2, C19.2, C2.2, C20.2, C23.1, C23.2, C24.1, C24.2, C25.1, C28.1, C28.2, C29.1, C29.2, C3.1, C3.2, C30.1, C31.1, C31.2, C4.1, C4.2, C5.1, C5.2, C6.2, C7.1, C7.2, C8.1, C8.2, C9.1, C9.2, D1.1 (K), D1.2 (A), D2.1 (K), J1.2 (Pin_2), J10.4 (Pin_4), J11.4 (Pin_4), J12.2 (Pin_2), J13.2 (Pin_2), J14.2 (Pin_2), J2.A1 (GND), J2.A12 (GND), J2.B1 (GND), J2.B12 (GND), J2.S1 (SHIELD), J7.1 (Pin_1), J7.2 (Pin_2), J8.1 (Pin_1), J8.2 (Pin_2), J9.1 (Pin_1), J9.2 (Pin_2), L1.1, L1.2, R1.2, R10.2, R11.2, R12.2, R13.2, R14.2, R15.2, R16.2, R17.2, R18.2, R19.2, R2.2, R20.2, R21.2, R3.2, R4.2, R6.2, R7.2, R8.2, R9.2, SW1.2, SW2.2, U1.2 (OUT), U1.3 (GND), U1.4 (FB), U1.5 (~{ON}/OFF), U2.1 (GND), U2.2 (VO), U2.3 (VI), U3.1 (GND), U3.2 (3V3), U3.40 (GND), U3.41 (GND), U4.10 (MS2/AD1), U4.13 (CLK), U4.15 (VCC_IO), U4.18 (GND), U4.22 (VS), U4.28 (VS), U4.29 (GND), U4.3 (GND), U4.7 (SPREAD), U4.8 (5VOUT), U4.9 (MS1/AD0), U5.10 (MS2/AD1), U5.13 (CLK), U5.15 (VCC_IO), U5.18 (GND), U5.29 (GND), U5.3 (GND), U5.7 (SPREAD), U5.8 (5VOUT), U5.9 (MS1/AD0), U6.10 (MS2/AD1), U6.13 (CLK), U6.15 (VCC_IO), U6.18 (GND), U6.29 (GND), U6.3 (GND), U6.7 (SPREAD), U6.8 (5VOUT), U6.9 (MS1/AD0), U7.10 (MS2/AD1), U7.13 (CLK), U7.15 (VCC_IO), U7.18 (GND), U7.29 (GND), U7.3 (GND), U7.7 (SPREAD), U7.8 (5VOUT), U7.9 (MS1/AD0), U8.1 (A0), U8.12 (GND), U8.2 (A1), U8.21 (A2), U8.24 (VCC), U8.3 (~{RESET})
- new net: C12.2, C14.1, C15.1, U4.22 (VS), U4.28 (VS)
- new net +3V3: C10.1, C31.1, C5.1, C7.1, C8.1, C9.1, J7.1 (Pin_1), J8.1 (Pin_1), J9.1 (Pin_1), R1.2, R14.2, R15.2, R16.2, R17.2, R18.2, R19.2, R2.2, R20.2, R21.2, U2.2 (VO), U3.2 (3V3), U4.15 (VCC_IO), U5.15 (VCC_IO), U5.9 (MS1/AD0), U6.10 (MS2/AD1), U6.15 (VCC_IO), U7.10 (MS2/AD1), U7.15 (VCC_IO), U7.9 (MS1/AD0), U8.24 (VCC), U8.3 (~{RESET})
- new net +5V: C3.1, C4.1, D2.1 (K), L1.1, U1.4 (FB), U2.3 (VI)
- new net 5VOUT_Pan: C18.1, U5.8 (5VOUT)
- new net 5VOUT_Slide: C13.1, U4.8 (5VOUT)
- new net 5VOUT_Tilt: C23.2, U6.8 (5VOUT)
- new net 5VOUT_Z: C28.2, U7.8 (5VOUT)
- new net GND: C1.2, C10.2, C14.2, C15.2, C18.2, C2.2, C20.2, C3.2, C31.2, C4.2, C5.2, C6.2, C7.2, C8.2, C9.2, D1.2 (A), J1.2 (Pin_2), J10.4 (Pin_4), J11.4 (Pin_4), J12.2 (Pin_2), J13.2 (Pin_2), J14.2 (Pin_2), J2.A1 (GND), J2.A12 (GND), J2.B1 (GND), J2.B12 (GND), J2.S1 (SHIELD), J7.2 (Pin_2), J8.2 (Pin_2), J9.2 (Pin_2), L1.2, R10.2, R11.2, R12.2, R13.2, R3.2, R4.2, R6.2, R7.2, R8.2, R9.2, SW1.2, SW2.2, U1.2 (OUT), U1.3 (GND), U1.5 (~{ON}/OFF), U2.1 (GND), U3.1 (GND), U3.40 (GND), U3.41 (GND), U4.10 (MS2/AD1), U4.13 (CLK), U4.18 (GND), U4.29 (GND), U4.3 (GND), U4.7 (SPREAD), U4.9 (MS1/AD0), U5.10 (MS2/AD1), U5.13 (CLK), U5.18 (GND), U5.29 (GND), U5.3 (GND), U5.7 (SPREAD), U6.13 (CLK), U6.18 (GND), U6.29 (GND), U6.3 (GND), U6.7 (SPREAD), U6.9 (MS1/AD0), U7.13 (CLK), U7.18 (GND), U7.29 (GND), U7.3 (GND), U7.7 (SPREAD), U8.1 (A0), U8.12 (GND), U8.2 (A1), U8.21 (A2)
Other:
- moved on the sheet: C10, C3, L1, R1, R2

Commit message: integrated pcb steppers done
Parts:
- removed C1, C15, C20, C25, C30: 100uF_35V, Capacitor_THT:CP_Radial_D8.0mm_P3.50mm, symbol Device:C_Polarized
- removed C10: 10uF, Capacitor_SMD:C_0805_2012Metric, symbol Device:C
- removed C11, C16, C21, C26: 22nF, Capacitor_SMD:C_0603_1608Metric, symbol Device:C
- removed C12, C14, C17, C19, C2, C22, C24, C27, C29, C31, C7, C8, C9: 100nF, Capacitor_SMD:C_0603_1608Metric, symbol Device:C
- removed C13, C18, C23, C28: 4.7uF, Capacitor_SMD:C_0603_1608Metric, symbol Device:C
- removed C3: 220uF_25V, Capacitor_THT:CP_Radial_D8.0mm_P3.50mm, symbol Device:C_Polarized
- removed C4: 10uF, Capacitor_SMD:C_0603_1608Metric, symbol Device:C
- removed C5: 22uF, Capacitor_SMD:C_0603_1608Metric, symbol Device:C
- removed C6: 1uF, Capacitor_SMD:C_0603_1608Metric, symbol Device:C
- removed D1: SS34, Diode_SMD:D_SMC, symbol Device:D_Schottky
- removed D2: SS14, Diode_SMD:D_SOD-123, symbol Device:D_Schottky
- removed F1: 2A, Fuse:Fuseholder_Clip-5x20mm_Littelfuse_111_Inline_P20.00x5.00mm_D1.05mm_Horizontal, symbol Device:Fuse
- removed J1: 24V_In, TerminalBlock:TerminalBlock_MaiXu_MX126-5.0-02P_1x02_P5.00mm, symbol Connector:Screw_Terminal_01x02
- removed J10: Enc_Jog, Connector_JST:JST_XH_B4B-XH-A_1x04_P2.50mm_Vertical, symbol Connector:Conn_01x04_Pin
- removed J11: Enc_Angle, Connector_JST:JST_XH_B4B-XH-A_1x04_P2.50mm_Vertical, symbol Connector:Conn_01x04_Pin
- removed J12: Limit_Min, Connector_JST:JST_XH_B2B-XH-A_1x02_P2.50mm_Vertical, symbol Connector:Conn_01x02_Pin
- removed J13: Limit_Max, Connector_JST:JST_XH_B2B-XH-A_1x02_P2.50mm_Vertical, symbol Connector:Conn_01x02_Pin
- removed J14: Limit_Z_Home, Connector_JST:JST_XH_B2B-XH-A_1x02_P2.50mm_Vertical, symbol Connector:Conn_01x02_Pin
- removed J2: USB_PROG, Connector_USB:USB_C_Receptacle_GCT_USB4085, symbol Connector:USB_C_Receptacle_USB2.0_14P
- removed J3: Motor_Slide, Connector_JST:JST_XH_B4B-XH-A_1x04_P2.50mm_Vertical, symbol Connector:Conn_01x04_Pin
- removed J4: Motor_Pan, Connector_JST:JST_XH_B4B-XH-A_1x04_P2.50mm_Vertical, symbol Connector:Conn_01x04_Pin
- removed J5: Motor_Tilt, Connector_JST:JST_XH_B4B-XH-A_1x04_P2.50mm_Vertical, symbol Connector:Conn_01x04_Pin
- removed J6: Motor_Z, Connector_JST:JST_XH_B4B-XH-A_1x04_P2.50mm_Vertical, symbol Connector:Conn_01x04_Pin
- removed J7: AS5600_Pan, Connector_JST:JST_XH_B4B-XH-A_1x04_P2.50mm_Vertical, symbol Connector:Conn_01x04_Pin
- removed J8: AS5600_Tilt, Connector_JST:JST_XH_B4B-XH-A_1x04_P2.50mm_Vertical, symbol Connector:Conn_01x04_Pin
- removed J9: OLED, Connector_JST:JST_XH_B4B-XH-A_1x04_P2.50mm_Vertical, symbol Connector:Conn_01x04_Pin
- removed L1: 100uH, Inductor_SMD:L_Bourns-SRN8040_8x8.15mm, symbol Device:L
- removed R1, R2: 10k, Resistor_SMD:R_0603_1608Metric, symbol Device:R
- removed R10, R11, R12, R13, R6, R7, R8, R9: 0.11, Resistor_SMD:R_0603_1608Metric, symbol Device:R
- removed R14, R15, R16, R17, R18, R19, R20, R21: 4.7k, Resistor_SMD:R_0603_1608Metric, symbol Device:R
- removed R3, R4: 5.1k, Resistor_SMD:R_0603_1608Metric, symbol Device:R
- removed R5: 1k, Resistor_SMD:R_0603_1608Metric, symbol Device:R
- removed SW1: BOOT, Button_Switch_THT:SW_PUSH_6mm, symbol Switch:SW_Push
- removed SW2: RESET, Button_Switch_THT:SW_PUSH_6mm, symbol Switch:SW_Push
- removed U1: LM2596S-5, Package_TO_SOT_SMD:TO-263-5_TabPin3, symbol Regulator_Switching:LM2596S-5
- removed U2: AMS1117-3.3, Package_TO_SOT_SMD:SOT-223-3_TabPin2, symbol Regulator_Linear:AMS1117-3.3
- removed U3: ESP32-S3-WROOM-1-N16R8, RF_Module:ESP32-S3-WROOM-1, symbol New_Library:ESP32-S3-WROOM-1
- removed U4, U5, U6, U7: TMC2209-LA, Package_DFN_QFN:VQFN-28-1EP_5x5mm_P0.5mm_EP3.7x3.7mm_ThermalVias, symbol Driver_Motor:TMC2209-LA
- removed U8: TCA9548APWR, Package_SO:TSSOP-24_4.4x7.8mm_P0.65mm, symbol Interface_Expansion:TCA9548APWR
Connections:
- no-connect marks 41 -> 0
Other:
- added sheet I2C-IO (I2C-IO.kicad_sch)
- added sheet esp32 (esp32.kicad_sch)
- added sheet power (power.kicad_sch)
- added sheet stepper drivers (untitled.kicad_sch)
- added sheet usb (usb.kicad_sch)
- note removed: "I2C MUX + OFF-BOARD I/O CONNECTORS"
- note removed: "MCU ESP32-S3-WROOM-1 + USB-C"
- note removed: "POWER 24V IN / 5V BUCK / 3V3 LDO"
- note removed: "STEPPER DRIVERS 4x TMC2209"
