File: integrated/schematic/untitled.kicad_sch (KiCad schematic)
At the start: 40 parts, among them J100 Motor_Slide, J101 Motor_Pan, J102 Motor_Tilt, J103 Motor_Z, U100 TMC2209-LA, U110 TMC2209-LA, U120 TMC2209-LA, U130 TMC2209-LA

Commit message: integrated pcb steppers done
Parts:
- removed C100, C110, C120, C130: 100uF_35V, Capacitor_THT:CP_Radial_D8.0mm_P3.50mm, symbol Device:C_Polarized
- removed C101, C102, C103, C111, C112, C113, C121, C122, C123, C131, C132, C133: 100nF, Capacitor_SMD:C_0603_1608Metric, symbol Device:C
- removed C104, C114, C124, C134: 4.7uF, Capacitor_SMD:C_0603_1608Metric, symbol Device:C
- removed C105, C115, C125, C135: 22nF, Capacitor_SMD:C_0603_1608Metric, symbol Device:C
- removed J100: Motor_Slide, Connector_JST:JST_XH_B4B-XH-A_1x04_P2.50mm_Vertical, symbol Connector:Conn_01x04_Pin
- removed J101: Motor_Pan, Connector_JST:JST_XH_B4B-XH-A_1x04_P2.50mm_Vertical, symbol Connector:Conn_01x04_Pin
- removed J102: Motor_Tilt, Connector_JST:JST_XH_B4B-XH-A_1x04_P2.50mm_Vertical, symbol Connector:Conn_01x04_Pin
- removed J103: Motor_Z, Connector_JST:JST_XH_B4B-XH-A_1x04_P2.50mm_Vertical, symbol Connector:Conn_01x04_Pin
- removed R100, R101, R110, R111, R120, R121, R130, R131: 0.11, Resistor_SMD:R_0603_1608Metric, symbol Device:R
- removed U100, U110, U120, U130: TMC2209-LA, Package_DFN_QFN:VQFN-28-1EP_5x5mm_P0.5mm_EP3.7x3.7mm_ThermalVias, symbol Driver_Motor:TMC2209-LA
- added C57, C58, C61, C62, C63, C64, C69, C70, C71, C74, C75, C76: 100nF, Capacitor_SMD:C_0603_1608Metric, symbol Device:C
- added C59, C60, C72, C73: 100uF_35V, Capacitor_THT:CP_Radial_D8.0mm_P3.50mm, symbol Device:C_Polarized
- added C65, C66, C77, C80: 4.7uF, Capacitor_SMD:C_0603_1608Metric, symbol Device:C
- added C67, C68, C78, C79: 22nF, Capacitor_SMD:C_0603_1608Metric, symbol Device:C
- added J27: Motor_Slide, Connector_JST:JST_XH_B4B-XH-A_1x04_P2.50mm_Vertical, symbol Connector:Conn_01x04_Pin
- added J28: Motor_Tilt, Connector_JST:JST_XH_B4B-XH-A_1x04_P2.50mm_Vertical, symbol Connector:Conn_01x04_Pin
- added J29: Motor_Pan, Connector_JST:JST_XH_B4B-XH-A_1x04_P2.50mm_Vertical, symbol Connector:Conn_01x04_Pin
- added J30: Motor_Z, Connector_JST:JST_XH_B4B-XH-A_1x04_P2.50mm_Vertical, symbol Connector:Conn_01x04_Pin
- added R38, R39, R40, R41, R42, R43, R44, R45: 0.11, Resistor_SMD:R_0603_1608Metric, symbol Device:R
- added U14, U15, U16, U17: TMC2209-LA, Package_DFN_QFN:VQFN-28-1EP_5x5mm_P0.5mm_EP3.7x3.7mm_ThermalVias, symbol Driver_Motor:TMC2209-LA
Connections:
- net +24V: now also C57.1, C58.1, C59.1, C60.1, C63.1, C64.1, C70.1, C71.1, C72.1, C73.1, C75.1, C76.1, U14.22 (VS), U14.28 (VS), U15.22 (VS), U15.28 (VS), U16.22 (VS), U16.28 (VS), U17.22 (VS), U17.28 (VS)
- net +3V3: now also C61.1, C62.1, C69.1, C74.1, U14.15 (VCC_IO), U15.10 (MS2/AD1), U15.15 (VCC_IO), U16.15 (VCC_IO), U16.9 (MS1/AD0), U17.10 (MS2/AD1), U17.15 (VCC_IO), U17.9 (MS1/AD0)
- net DIAG0: now also U14.11 (DIAG)
- net DIAG1: now also U16.11 (DIAG)
- net DIAG2: now also U15.11 (DIAG)
- net DIAG3: now also U17.11 (DIAG)
- net DIR0: now also U14.19 (DIR)
- net DIR1: now also U16.19 (DIR)
- net DIR2: now also U15.19 (DIR)
- net DIR3: now also U17.19 (DIR)
- net EN: now also U14.2 (~{EN}), U15.2 (~{EN}), U16.2 (~{EN}), U17.2 (~{EN})
- net GND: now also C57.2, C58.2, C59.2, C60.2, C61.2, C62.2, C65.1, C66.2, C69.2, C70.2, C71.2, C72.2, C73.2, C74.2, C77.1, C80.1, R38.2, R39.2, R40.2, R41.2, R42.2, R43.2, R44.2, R45.2, U14.10 (MS2/AD1), U14.13 (CLK), U14.18 (GND), U14.20 (STDBY), U14.29 (GND), U14.3 (GND), U14.7 (SPREAD), U14.9 (MS1/AD0), U15.13 (CLK), U15.18 (GND), U15.20 (STDBY), U15.29 (GND), U15.3 (GND), U15.7 (SPREAD), U15.9 (MS1/AD0), U16.10 (MS2/AD1), U16.13 (CLK), U16.18 (GND), U16.20 (STDBY), U16.29 (GND), U16.3 (GND), U16.7 (SPREAD), U17.13 (CLK), U17.18 (GND), U17.20 (STDBY), U17.29 (GND), U17.3 (GND), U17.7 (SPREAD)
- net M0_A1: now also J27.1 (Pin_1), U14.24 (OA1)
- net M0_A2: now also J27.2 (Pin_2), U14.21 (OA2)
- net M0_B1: now also J27.3 (Pin_3), U14.26 (OB1)
- net M0_B2: now also J27.4 (Pin_4), U14.1 (OB2)
- net M1_A1: now also J29.1 (Pin_1), U16.24 (OA1)
- net M1_A2: now also J29.2 (Pin_2), U16.21 (OA2)
- net M1_B1: now also J29.3 (Pin_3), U16.26 (OB1)
- net M1_B2: now also J29.4 (Pin_4), U16.1 (OB2)
- net M2_A1: now also J28.1 (Pin_1), U15.24 (OA1)
- net M2_A2: now also J28.2 (Pin_2), U15.21 (OA2)
- net M2_B1: now also J28.3 (Pin_3), U15.26 (OB1)
- net M2_B2: now also J28.4 (Pin_4), U15.1 (OB2)
- net M3_A1: now also J30.1 (Pin_1), U17.24 (OA1)
- net M3_A2: now also J30.2 (Pin_2), U17.21 (OA2)
- net M3_B1: now also J30.3 (Pin_3), U17.26 (OB1)
- net M3_B2: now also J30.4 (Pin_4), U17.1 (OB2)
- net STEP0: now also U14.16 (STEP)
- net STEP1: now also U16.16 (STEP)
- net STEP2: now also U15.16 (STEP)
- net STEP3: now also U17.16 (STEP)
- net UART: now also U14.14 (~{PD}/UART), U15.14 (~{PD}/UART), U16.14 (~{PD}/UART), U17.14 (~{PD}/UART)
- new net: C64.2, U15.6 (VCP)
- new net: C77.2, U16.8 (5VOUT)
- new net: R40.1, U14.23 (BRA)
- new net: R38.1, U14.27 (BRB)
- new net: C67.1, U14.4 (CPO)
- new net: C67.2, U14.5 (CPI)
- new net: C63.2, U14.6 (VCP)
- new net: C65.2, U14.8 (5VOUT)
- new net: R43.1, U17.27 (BRB)
- new net: R41.1, U15.23 (BRA)
- new net: R39.1, U15.27 (BRB)
- new net: C68.1, U15.4 (CPO)
- new net: C68.2, U15.5 (CPI)
- new net: C66.1, U15.8 (5VOUT)
- new net: R42.1, U16.27 (BRB)
- new net: R45.1, U17.23 (BRA)
- new net: R44.1, U16.23 (BRA)
- new net: C78.1, U16.4 (CPO)
- new net: C78.2, U16.5 (CPI)
- new net: C75.2, U16.6 (VCP)
- new net: C76.2, U17.6 (VCP)
- new net: C79.1, U17.4 (CPO)
- new net: C79.2, U17.5 (CPI)
- new net: C80.2, U17.8 (5VOUT)
Other:
- title: PanTilt Slide -- Stepper Drivers (integrated TMC2209-LA) -> (none)
