File: hybrid/schematic/tmc2209_driver_stepstick.kicad_sch (KiCad schematic)
At the start: 24 parts, among them J100 Motor_Slide, J101 Motor_Pan, J102 Motor_Tilt, J103 Motor_Z, J110 PDN_DIAG_0, J111 PDN_DIAG_1, J112 PDN_DIAG_2, J113 PDN_DIAG_3

Commit message: fullpcb filled out
Parts:
- removed A100, A110, A120, A130: TMC2209_StepStick, Module:Pololu_Breakout-16_15.2x20.3mm, symbol Driver_Motor:Pololu_Breakout_A4988
- removed C100, C110, C120, C130: 100uF_35V, Capacitor_THT:CP_Radial_D8.0mm_P3.50mm, symbol Device:C_Polarized
- removed C101, C102, C111, C112, C121, C122, C131, C132: 100nF, Capacitor_SMD:C_0603_1608Metric, symbol Device:C
- removed J100: Motor_Slide, Connector_JST:JST_XH_B4B-XH-A_1x04_P2.50mm_Vertical, symbol Connector:Conn_01x04_Pin
- removed J101: Motor_Pan, Connector_JST:JST_XH_B4B-XH-A_1x04_P2.50mm_Vertical, symbol Connector:Conn_01x04_Pin
- removed J102: Motor_Tilt, Connector_JST:JST_XH_B4B-XH-A_1x04_P2.50mm_Vertical, symbol Connector:Conn_01x04_Pin
- removed J103: Motor_Z, Connector_JST:JST_XH_B4B-XH-A_1x04_P2.50mm_Vertical, symbol Connector:Conn_01x04_Pin
- removed J110: PDN_DIAG_0, Connector_PinHeader_2.54mm:PinHeader_1x02_P2.54mm_Vertical, symbol Connector:Conn_01x02_Pin
- removed J111: PDN_DIAG_1, Connector_PinHeader_2.54mm:PinHeader_1x02_P2.54mm_Vertical, symbol Connector:Conn_01x02_Pin
- removed J112: PDN_DIAG_2, Connector_PinHeader_2.54mm:PinHeader_1x02_P2.54mm_Vertical, symbol Connector:Conn_01x02_Pin
- removed J113: PDN_DIAG_3, Connector_PinHeader_2.54mm:PinHeader_1x02_P2.54mm_Vertical, symbol Connector:Conn_01x02_Pin
- added U3, U5, U6, U7: tmc2209, TMC2209:TMC2209_SilentStepStick_Socket_18P, symbol New_Library:tmc2209
Connections:
- net +24V: now also U3.8 (VM), U5.8 (VM), U6.8 (VM), U7.8 (VM)
- net GND: now also U3.1 (GND), U3.14 (MS2), U3.15 (MS1), U3.7 (GND), U5.1 (GND), U5.14 (MS2), U5.7 (GND), U6.1 (GND), U6.15 (MS1), U6.7 (GND), U7.1 (GND), U7.7 (GND)
- new net 3.3v: U3.2 (VIO), U5.15 (MS1), U5.2 (VIO), U6.14 (MS2), U6.2 (VIO), U7.14 (MS2), U7.15 (MS1), U7.2 (VIO)
- new net AUX_M1A: U7.4 (M1A)
- new net AUX_M1B: U7.3 (M1B)
- new net AUX_M2A: U7.5 (M2A)
- new net AUX_M2B: U7.6 (M2B)
- new net GPIO_10: U3.16 (En), U5.16 (En), U6.16 (En), U7.16 (En)
- new net GPIO_4: U3.10 (Step)
- new net GPIO_41: U3.12 (UART), U5.12 (UART), U6.12 (UART), U7.12 (UART)
- new net GPIO_42: U3.11 (PDN), U5.11 (PDN), U6.11 (PDN), U7.11 (PDN)
- new net GPIO_47: U7.10 (Step)
- new net GPIO_48: U7.9 (DIR)
- new net GPIO_5: U3.9 (DIR)
- new net GPIO_6: U5.10 (Step)
- new net GPIO_7: U5.9 (DIR)
- new net GPIO_8: U6.10 (Step)
- new net GPIO_9: U6.9 (DIR)
- new net PAN_M1A: U5.4 (M1A)
- new net PAN_M1B: U5.3 (M1B)
- new net PAN_M2A: U5.5 (M2A)
- new net PAN_M2B: U5.6 (M2B)
- new net SLIDE_M1A: U3.4 (M1A)
- new net SLIDE_M1B: U3.3 (M1B)
- new net SLIDE_M2A: U3.5 (M2A)
- new net SLIDE_M2B: U3.6 (M2B)
- new net TILT_M1A: U6.4 (M1A)
- new net TILT_M1B: U6.3 (M1B)
- new net TILT_M2A: U6.5 (M2A)
- new net TILT_M2B: U6.6 (M2B)
- no-connect marks 8 -> 12
Other:
- note removed: "1 -> module PDN_UART pad 2 -> module DIAG pad"
- note removed: "Drop-in alternative to tmc2209_driver_chip.kicad_sch -- identical sheet pins."
- note removed: "STEPPER 0 (Slide) UART addr 0"
- note removed: "STEPPER 1 (Pan) UART addr 1"
- note removed: "STEPPER 2 (Tilt) UART addr 2"
- note removed: "STEPPER 3 (Z) UART addr 3"
- note removed: "STEPPER DRIVERS -- 4 x plug-in TMC2209 StepStick"
- note removed: "Set motor current with the module trimpot (VREF); the module carries its own sense resistors, charge pump and 5V regulator."
- note removed: "Socket = Pololu / StepStick 2x8 outline, drawn with the A4988 legacy pin names. TMC2209 SilentStepStick function by pin number: 9=EN 10=MS1/AD0 11=MS2/AD1 12=SPREAD 13,14=no pin on the module 15=STEP 16=DIR 2=VIO 8=VM 1,7=GND 3=OB2 4=OB1 5=OA1 6=OA2."
