File: pantiltslide/pantiltslide_full.kicad_sch (KiCad schematic)
At the start: 31 parts, among them J1 Conn_01x22_Socket, J10 Conn_01x04_Pin, J11 Conn_01x04_Pin, J12 Conn_01x04_Pin, J13 Conn_01x04_Pin, J14 Conn_01x04_Pin, J15 Conn_01x04_Pin, J16 Conn_01x04_Pin, J17 Motor_Slide, J18 Motor_Pan, J19 Motor_Tilt, J2 Conn_01x22_Socket, J20 TCA9548A_Mux, J21 AS5600_Pan, J22 AS5600_Tilt, J23 OLED, J24 Jog_Encoder, J25 Manual_Setpoint_Encoder, J26 Limit_Min, J27 Limit_Max, J3 Conn_01x08_Socket, J4 Conn_01x08_Socket, J7 Conn_01x12_Socket, J8 Conn_01x12_Socket, J9 Conn_01x04_Pin, U1 tmc2209, U2 tmc2209, U3 tmc2209

Commit message: pcb updates
Parts:
- removed J24: Jog_Encoder, Connector_PinHeader_2.54mm:PinHeader_1x04_P2.54mm_Vertical, symbol Connector:Conn_01x04_Pin
- removed J25: Manual_Setpoint_Encoder, Connector_PinHeader_2.54mm:PinHeader_1x04_P2.54mm_Vertical, symbol Connector:Conn_01x04_Pin
- added J28: Motor_Aux, Connector_PinHeader_2.54mm:PinHeader_1x04_P2.54mm_Vertical, symbol Connector:Conn_01x04_Pin
- added J29: Enc_Slide, Connector_PinHeader_2.54mm:PinHeader_1x04_P2.54mm_Vertical, symbol Connector:Conn_01x04_Pin
- added J30: Enc_Pan, Connector_PinHeader_2.54mm:PinHeader_1x04_P2.54mm_Vertical, symbol Connector:Conn_01x04_Pin
- added J31: Enc_Tilt, Connector_PinHeader_2.54mm:PinHeader_1x04_P2.54mm_Vertical, symbol Connector:Conn_01x04_Pin
- added J32: Enc_Aux, Connector_PinHeader_2.54mm:PinHeader_1x04_P2.54mm_Vertical, symbol Connector:Conn_01x04_Pin
- added J33: Btn_SetKeyframe, TerminalBlock:TerminalBlock_MaiXu_MX126-5.0-02P_1x02_P5.00mm, symbol Connector:Screw_Terminal_01x02
- added J34: Btn_ClearKeyframe, TerminalBlock:TerminalBlock_MaiXu_MX126-5.0-02P_1x02_P5.00mm, symbol Connector:Screw_Terminal_01x02
- added J35: Btn_PlayPause, TerminalBlock:TerminalBlock_MaiXu_MX126-5.0-02P_1x02_P5.00mm, symbol Connector:Screw_Terminal_01x02
- added J36: Btn_Reset, TerminalBlock:TerminalBlock_MaiXu_MX126-5.0-02P_1x02_P5.00mm, symbol Connector:Screw_Terminal_01x02
- added U4: tmc2209, TMC2209:TMC2209_SilentStepStick_Socket_18P, symbol New_Library:tmc2209
- F1: footprint (none) -> Fuse:Fuseholder_Clip-5x20mm_Littelfuse_111_Inline_P20.00x5.00mm_D1.05mm_Horizontal
- J1, J2: footprint (none) -> Connector_PinSocket_2.54mm:PinSocket_1x22_P2.54mm_Vertical
- J10, J11, J12, J13, J14, J15, J16, J9: footprint (none) -> Connector_PinHeader_2.54mm:PinHeader_1x04_P2.54mm_Vertical
- J26, J27: footprint TerminalBlock_MaiXu:TerminalBlock_MaiXu_MX126-5.0-02P_1x02_P5.00mm -> TerminalBlock:TerminalBlock_MaiXu_MX126-5.0-02P_1x02_P5.00mm
- J3, J4: footprint (none) -> Connector_PinSocket_2.54mm:PinSocket_1x08_P2.54mm_Vertical
- J37: renamed from 5Vin; value Screw_Terminal_01x02 -> 5V_In; footprint (none) -> TerminalBlock:TerminalBlock_MaiXu_MX126-5.0-02P_1x02_P5.00mm
- J38: renamed from 24Vin; value Screw_Terminal_01x02 -> 24V_In; footprint (none) -> TerminalBlock:TerminalBlock_MaiXu_MX126-5.0-02P_1x02_P5.00mm
- J7, J8: footprint (none) -> Connector_PinSocket_2.54mm:PinSocket_1x12_P2.54mm_Vertical
Connections:
- net +24V: now also U4.8 (VM)
- net +3.3V: now also U4.14 (MS2), U4.15 (MS1), U4.2 (VIO)
- net GND: now also J29.3 (Pin_3), J30.3 (Pin_3), J31.3 (Pin_3), J32.3 (Pin_3), J33.2 (Pin_2), J34.2 (Pin_2), J35.2 (Pin_2), J36.2 (Pin_2), U4.1 (GND), U4.7 (GND)
- net GPIO_1: now also J33.1 (Pin_1)
- net GPIO_10: now also U4.16 (En)
- net GPIO_15: now also J29.1 (Pin_1)
- net GPIO_16: now also J29.2 (Pin_2)
- net GPIO_17: now also J30.1 (Pin_1)
- net GPIO_18: now also J30.2 (Pin_2)
- net GPIO_19: now also J32.1 (Pin_1)
- net GPIO_20: now also J32.2 (Pin_2)
- net GPIO_21: now also J31.1 (Pin_1)
- net GPIO_3: now also J34.1 (Pin_1)
- net GPIO_38: now also J31.2 (Pin_2)
- net GPIO_41: now also U4.12 (UART)
- net GPIO_42: now also U4.11 (PDN)
- net GPIO_45: now also J35.1 (Pin_1)
- net GPIO_46: now also J36.1 (Pin_1)
- net GPIO_47: now also U4.10 (Step)
- net GPIO_48: now also U4.9 (DIR)
- new net AUX_M1A: J28.1 (Pin_1), U4.4 (M1A)
- new net AUX_M1B: J28.2 (Pin_2), U4.3 (M1B)
- new net AUX_M2A: J28.3 (Pin_3), U4.5 (M2A)
- new net AUX_M2B: J28.4 (Pin_4), U4.6 (M2B)
- no-connect marks 9 -> 16

Commit message: fullpcb filled out
Parts:
- removed J10, J11, J12, J13, J14, J15, J16, J9: Conn_01x04_Pin, Connector_PinHeader_2.54mm:PinHeader_1x04_P2.54mm_Vertical, symbol Connector:Conn_01x04_Pin
- removed J3, J4: Conn_01x08_Socket, Connector_PinSocket_2.54mm:PinSocket_1x08_P2.54mm_Vertical, symbol Connector:Conn_01x08_Socket
- removed J7, J8: Conn_01x12_Socket, Connector_PinSocket_2.54mm:PinSocket_1x12_P2.54mm_Vertical, symbol Connector:Conn_01x12_Socket
- added J24: TCA9548A_Mux, Connector_PinSocket_2.54mm:PinSocket_1x12_P2.54mm_Vertical, symbol Connector:Conn_01x12_Socket
- J17, J18, J19, J21, J22, J28: footprint Connector_PinHeader_2.54mm:PinHeader_1x04_P2.54mm_Vertical -> Connector_JST:JST_XH_B4B-XH-A_1x04_P2.50mm_Vertical
- J20: footprint Connector_PinSocket_2.54mm:PinSocket_1x08_P2.54mm_Vertical -> Connector_PinSocket_2.54mm:PinSocket_1x12_P2.54mm_Vertical; symbol Connector:Conn_01x08_Socket -> Connector:Conn_01x12_Socket
- J26, J27, J33, J34, J35, J36: footprint TerminalBlock:TerminalBlock_MaiXu_MX126-5.0-02P_1x02_P5.00mm -> Connector_JST:JST_XH_B2B-XH-A_1x02_P2.50mm_Vertical; symbol Connector:Screw_Terminal_01x02 -> Connector_Generic:Conn_01x02
- J29, J30, J31, J32: footprint Connector_PinHeader_2.54mm:PinHeader_1x04_P2.54mm_Vertical -> JST_EH_B3B-EH-A_1x03_P2.50mm_Vertical; symbol Connector:Conn_01x04_Pin -> Connector_Generic:Conn_01x03
Connections:
- net +3.3V: now also J20.5 (Pin_5)
- net GND: now also J20.6 (Pin_6), J20.7 (Pin_7), J20.8 (Pin_8)
- net GPIO_1: no longer J2.5 (Pin_5)
- net MUX_CH0_SCL: now also J20.10 (Pin_10); no longer J20.6 (Pin_6)
- net MUX_CH0_SDA: now also J20.9 (Pin_9); no longer J20.5 (Pin_5)
- net MUX_CH1_SCL: now also J20.12 (Pin_12); no longer J20.8 (Pin_8)
- net MUX_CH1_SDA: now also J20.11 (Pin_11); no longer J20.7 (Pin_7)
- new net GPIO_2: J2.5 (Pin_5)
- new net MUX_CH2_SCL: J24.12 (Pin_12)
- new net MUX_CH2_SDA: J24.11 (Pin_11)
- new net MUX_CH3_SCL: J24.10 (Pin_10)
- new net MUX_CH3_SDA: J24.9 (Pin_9)
- new net MUX_CH4_SCL: J24.8 (Pin_8)
- new net MUX_CH4_SDA: J24.7 (Pin_7)
- new net MUX_CH5_SCL: J24.6 (Pin_6)
- new net MUX_CH5_SDA: J24.5 (Pin_5)
- new net MUX_CH6_SCL: J24.4 (Pin_4)
- new net MUX_CH6_SDA: J24.3 (Pin_3)
- new net MUX_CH7_SCL: J24.2 (Pin_2)
- new net MUX_CH7_SDA: J24.1 (Pin_1)
- no-connect marks 16 -> 12
