File: pantiltslide/pantiltslide_full_pwr.kicad_pcb (KiCad board)
At the start: 4 copper layers, 76 x 113 mm, 28 parts, among them J1 Conn_01x22_Socket, J17 Motor_Slide, J18 Motor_Pan, J19 Motor_Tilt, J2 Conn_01x22_Socket, J20 TCA9548A_Mux, J21 AS5600_Pan, J22 AS5600_Tilt, J23 OLED, J24 TCA9548A_Mux, J26 Limit_Min, J27 Limit_Max, J28 Motor_Aux, J29 Enc_Slide, J30 Enc_Pan, J31 Enc_Tilt, J32 Enc_Aux, J33 Btn_SetKeyframe, J34 Btn_ClearKeyframe, J35 Btn_PlayPause, J36 Btn_Reset, J37 5V_In, J38 24V_In, U1 tmc2209, U2 tmc2209, U3 tmc2209, U4 tmc2209

Commit message: updates and corrections
Parts:
- added C1: 470uF/50V, Capacitor_THT:CP_Radial_D10.0mm_P5.00mm, F.Cu at (190.2, 27.3)
- added C2: 100nF/50V, Capacitor_SMD:C_0805_2012Metric, F.Cu at (202.7, 23.0)
- added C3: 220uF/25V, Capacitor_THT:CP_Radial_D8.0mm_P3.50mm, F.Cu at (179.5, 54.3)
- added C4: 10uF, Capacitor_SMD:C_0805_2012Metric, F.Cu at (203.2, 51.0)
- added C5: 22uF, Capacitor_SMD:C_0805_2012Metric, F.Cu at (178.7, 62.6)
- added C6: 100nF, Capacitor_SMD:C_0805_2012Metric, F.Cu at (185.2, 62.6)
- added D1: SS34, Diode_SMD:D_SMC, F.Cu at (213.5, 39.0)
- added D2: SS34, Diode_SMD:D_SMC, F.Cu at (193.5, 53.4)
- added D3: SMBJ33A, Diode_SMD:D_SMB, F.Cu at (180.7, 24.3)
- added D4: LED_24V, LED_SMD:LED_0805_2012Metric, F.Cu at (215.6, 23.0)
- added D5: LED_3V3, LED_SMD:LED_0805_2012Metric, F.Cu at (198.2, 62.6)
- added JP1: 0R, Resistor_SMD:R_0805_2012Metric, F.Cu at (204.6, 62.6)
- added L1: 100uH/3A, Inductor_SMD:L_Bourns-SRN8040_8x8.15mm, F.Cu at (201.1, 40.0)
- added R1: 10k, Resistor_SMD:R_0805_2012Metric, F.Cu at (209.2, 23.0)
- added R10: 2.2k, Resistor_SMD:R_0805_2012Metric, F.Cu at (178.7, 72.6)
- added R2: 1k, Resistor_SMD:R_0805_2012Metric, F.Cu at (191.7, 62.6)
- added R3: 4.7k, Resistor_SMD:R_0805_2012Metric, F.Cu at (211.1, 62.6)
- added R4: 4.7k, Resistor_SMD:R_0805_2012Metric, F.Cu at (178.7, 67.6)
- added R5: 4.7k, Resistor_SMD:R_0805_2012Metric, F.Cu at (185.2, 67.6)
- added R6: 4.7k, Resistor_SMD:R_0805_2012Metric, F.Cu at (191.6, 67.6)
- added R7: 2.2k, Resistor_SMD:R_0805_2012Metric, F.Cu at (198.1, 67.6)
- added R8: 2.2k, Resistor_SMD:R_0805_2012Metric, F.Cu at (204.5, 67.6)
- added R9: 2.2k, Resistor_SMD:R_0805_2012Metric, F.Cu at (211.0, 67.6)
- added U5: LM2596S-5, Package_TO_SOT_SMD:TO-263-5_TabPin3, F.Cu at (187.2, 41.3)
- added U6: AMS1117-3.3, Package_TO_SOT_SMD:SOT-223-3_TabPin2, F.Cu at (212.4, 53.6)
Connections:
- J1 pad 1: 3.3v -> ESP_3V3
- J1 pad 2: 3.3v -> ESP_3V3
Routing:
- net 3.3v: track 298.2 -> 262.4 mm
- net ESP_3V3: track 0.00 -> 2.54 mm
Other:
- board size 76 x 113 mm -> 123 x 113 mm
