File: pantiltslide/pantiltslide_full_turnkey.kicad_sch (KiCad schematic)
At the start: 53 parts, among them J1 Conn_01x22_Socket, J17 Motor_Slide, J18 Motor_Pan, J19 Motor_Tilt, J2 Conn_01x22_Socket, J20 TCA9548A_Mux, J21 AS5600_Pan, J22 AS5600_Tilt, J23 OLED, J24 TCA9548A_Mux, J26 Limit_Min, J27 Limit_Max, J28 Motor_Aux, J29 Enc_Slide, J30 Enc_Pan, J31 Enc_Tilt, J32 Enc_Aux, J33 Btn_SetKeyframe, J34 Btn_ClearKeyframe, J35 Btn_PlayPause, J36 Btn_Reset, J37 5V_In, J38 24V_In, U1 tmc2209, U2 tmc2209, U3 tmc2209, U4 tmc2209

Commit message: fixing uart, and adjusting pins
Parts:
- added J41: Aux_Max, Connector_JST:JST_XH_B2B-XH-A_1x02_P2.50mm_Vertical, symbol Connector_Generic:Conn_01x02
- added R10, R11: 100R, symbol Device:R
- added R9: 1k, PCM_SparkFun-Resistor:R_0402_1005Metric, symbol PCM_SparkFun-Resistor:1k_0402
- J29, J30, J31, J32: footprint JST_EH_B3B-EH-A_1x03_P2.50mm_Vertical -> Connector_JST:JST_XH_B3B-XH-A_1x03_P2.50mm_Vertical
- U4: footprint TMC2209:TMC2209_SilentStepStick_Socket_18P -> (none)
Connections:
- net GND: now also J41.2 (Pin_2)
- net GPIO_1: now also U4.10 (Step); no longer J33.1 (Pin_1)
- net GPIO_2: now also U4.9 (DIR)
- net GPIO_41: now also R10.1; no longer U1.12 (UART), U2.12 (UART), U3.12 (UART), U4.12 (UART)
- net GPIO_42: now also R11.1; no longer U1.11 (PDN), U2.11 (PDN), U3.11 (PDN), U4.11 (PDN)
- net GPIO_47: now also J33.1 (Pin_1); no longer U4.10 (Step)
- net GPIO_48: now also J41.1 (Pin_1); no longer U4.9 (DIR)
- new net: R10.2, R9.1
- new net UART: R11.2, R9.2, U1.11 (PDN), U2.11 (PDN), U3.11 (PDN), U4.11 (PDN)
- no-connect marks 12 -> 16
Other:
- moved on the sheet: U1, U2, U3, U4

Commit message: updates
Connections:
- net GPIO_41: now also R11.1; no longer R10.1
- net GPIO_42: now also J41.1 (Pin_1); no longer R11.1
- net GPIO_47: now also R10.1; no longer J33.1 (Pin_1)
- net GPIO_48: no longer J41.1 (Pin_1)
Other:
- note added: "RX"
- note added: "TX"
- moved on the sheet: J34, J35
Changed lines of the file:
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@@
 		)
 	)
+	(text "RX\n"
+		(exclude_from_sim no)
+		(at 299.974 296.418 0)
+		(effects
+			(font
+				(size 1.27 1.27)
+			)
+		)
+	)
+	(text "TX\n"
+		(exclude_from_sim no)
+		(at 300.228 291.338 0)
+		(effects
+			(font
+				(size 1.27 1.27)
+			)
+		)
+	)
 	(text "DECOUPLING  -  every cap carries a `Decouples` field naming the pin it belongs beside"
 		(exclude_from_sim no)
@@
 	(wire
 		(pts
-			(xy 514.92 280) (xy 507.3 280)
+			(xy 511.81 274.32) (xy 504.19 274.32)
 		)
 		(stroke
@@
 	(wire
 		(pts
-			(xy 514.92 245) (xy 507.3 245)
+			(xy 513.08 243.84) (xy 505.46 243.84)
 		)
 		(stroke
@@
 	(wire
 		(pts
-			(xy 514.92 282.54) (xy 507.3 282.54)
+			(xy 511.81 276.86) (xy 504.19 276.86)
 		)
 		(stroke
@@
 	(wire
 		(pts
-			(xy 514.92 247.54) (xy 507.3 247.54)
+			(xy 513.08 246.38) (xy 505.46 246.38)
 		)
 		(stroke
@@
 		)
 	)
-	(global_label "GPIO_41"
+	(global_label "GPIO_47"
 		(shape input)
 		(at 312.42 290.83 180)
@@
 		)
 	)
-	(global_label "GPIO_47"
-		(shape input)
-		(at 507.3 210 180)
-		(effects
-			(font
-				(size 1.27 1.27)
-			)
-			(justify right)
-		)
-		(property "Intersheetrefs" "${INTERSHEET_REFS}"
-			(at 507.3 210 0)
-			(hide yes)
-			(show_name no)
-			(do_not_autoplace no)
-			(effects
-				(font
-					(size 1.27 1.27)
-				)
-			)
-		)
-	)
 	(global_label "AUX_M2A"
 		(shape input)
@@
 		)
 	)
-	(global_label "UART"
+	(global_label "GPIO_3"
 		(shape input)
-		(at 332.74 290.83 0)
+		(at 505.46 243.84 180)
 		(effects
 			(font
 				(size 1.27 1.27)
 			)
-			(justify left)
+			(justify right)
 		)
 		(property "Intersheetrefs" "${INTERSHEET_REFS}"
-			(at 332.74 290.83 0)
+			(at 505.46 243.84 0)
 			(hide yes)
 			(show_name no)
@@
 		)
 	)
-	(global_label "SLIDE_M1B"
+	(global_label "UART"
 		(shape input)
-		(at 372.7 40 0)
+		(at 332.74 290.83 0)
 		(effects
 			(font
@@
 		)
 		(property "Intersheetrefs" "${INTERSHEET_REFS}"
-			(at 372.7 40 0)
+			(at 332.74 290.83 0)
 			(hide yes)
 			(show_name no)
@@
 		)
 	)
-	(global_label "GPIO_17"
+	(global_label "SLIDE_M1B"
 		(shape input)
-		(at 442.7 207.46 0)
+		(at 372.7 40 0)
 		(effects
 			(font
@@
 		)
 		(property "Intersheetrefs" "${INTERSHEET_REFS}"
-			(at 442.7 207.46 0)
+			(at 372.7 40 0)
 			(hide yes)
 			(show_name no)
@@
 		)
 	)
-	(global_label "GPIO_3"
+	(global_label "GPIO_17"
 		(shape input)
-		(at 507.3 245 180)
+		(at 442.7 207.46 0)
 		(effects
 			(font
 				(size 1.27 1.27)
 			)
-			(justify right)
+			(justify left)
 		)
 		(property "Intersheetrefs" "${INTERSHEET_REFS}"
-			(at 507.3 245 0)
+			(at 442.7 207.46 0)
 			(hide yes)
 			(show_name no)
@@
 		)
 	)
-	(global_label "GPIO_48"
+	(global_label "GPIO_42"
 		(shape input)
 		(at 506.73 184.15 180)
@@
 		)
 	)
+	(global_label "GPIO_45"
+		(shape input)
+		(at 504.19 274.32 180)
+		(effects
+			(font
+				(size 1.27 1.27)
+			)
+			(justify right)
+		)
+		(property "Intersheetrefs" "${INTERSHEET_REFS}"
+			(at 504.19 274.32 0)
+			(hide yes)
+			(show_name no)
+			(do_not_autoplace no)
+			(effects
+				(font
+					(size 1.27 1.27)
+				)
+			)
+		)
+	)
 	(global_label "GPIO_13"
 		(shape input)
@@
 		)
 	)
-	(global_label "GPIO_42"
+	(global_label "GPIO_41"
 		(shape input)
 		(at 312.42 295.91 180)
@@
 		)
 	)
-	(global_label "GPIO_45"
-		(shape input)
-		(at 507.3 280 180)
-		(effects
-			(font
-				(size 1.27 1.27)
-			)
-			(justify right)
-		)
-		(property "Intersheetrefs" "${INTERSHEET_REFS}"
-			(at 507.3 280 0)
-			(hide yes)
-			(show_name no)
-			(do_not_autoplace no)
-			(effects
-				(font
-					(size 1.27 1.27)
-				)
-			)
-		)
-	)
 	(global_label "GPIO_7"
 		(shape input)
@@
 	(global_label "GND"
 		(shape input)
-		(at 507.3 247.54 180)
+		(at 505.46 246.38 180)
 		(effects
 			(font
@@
 		)
 		(property "Intersheetrefs" "${INTERSHEET_REFS}"
-			(at 507.3 247.54 0)
+			(at 505.46 246.38 0)
 			(hide yes)
 			(show_name no)
@@
 	(global_label "GND"
 		(shape input)
-		(at 507.3 282.54 180)
+		(at 504.19 276.86 180)
 		(effects
 			(font
@@
 		)
 		(property "Intersheetrefs" "${INTERSHEET_REFS}"
-			(at 507.3 282.54 0)
+			(at 504.19 276.86 0)
 			(hide yes)
 			(show_name no)
@@
 	(symbol
 		(lib_id "Connector_Generic:Conn_01x02")
-		(at 520 245 0)
+		(at 518.16 243.84 0)
 		(unit 1)
 		(body_style 1)
@@
 		(fields_autoplaced yes)
 		(property "Reference" "J34"
-			(at 523.24 244.9999 0)
+			(at 521.4 243.8399 0)
 			(show_name no)
 			(do_not_autoplace no)
@@
 		)
 		(property "Value" "Btn_ClearKeyframe"
-			(at 523.24 247.5399 0)
+			(at 521.4 246.3799 0)
 			(show_name no)
 			(do_not_autoplace no)
@@
 		)
 		(property "Footprint" "Connector_JST:JST_XH_B2B-XH-A_1x02_P2.50mm_Vertical"
-			(at 520 245 0)
+			(at 518.16 243.84 0)
 			(hide yes)
 			(show_name no)
@@
 		)
 		(property "Datasheet" ""
-			(at 520 245 0)
+			(at 518.16 243.84 0)
 			(hide yes)
 			(show_name no)
@@
 		)
 		(property "Description" "Generic connector, single row, 01x02, script generated (kicad-library-utils/schlib/autogen/connector/)"
-			(at 520 245 0)
+			(at 518.16 243.84 0)
 			(hide yes)
 			(show_name no)
@@
 	(symbol
 		(lib_id "Connector_Generic:Conn_01x02")
-		(at 520 280 0)
+		(at 516.89 274.32 0)
 		(unit 1)
 		(body_style 1)
@@
 		(fields_autoplaced yes)
 		(property "Reference" "J35"
-			(at 523.24 279.9999 0)
+			(at 520.13 274.3199 0)
 			(show_name no)
 			(do_not_autoplace no)
@@
 		)
 		(property "Value" "Btn_PlayPause"
-			(at 523.24 282.5399 0)
+			(at 520.13 276.8599 0)
 			(show_name no)
 			(do_not_autoplace no)
@@
 		)
 		(property "Footprint" "Connector_JST:JST_XH_B2B-XH-A_1x02_P2.50mm_Vertical"
-			(at 520 280 0)
+			(at 516.89 274.32 0)
 			(hide yes)
 			(show_name no)
@@
 		)
 		(property "Datasheet" ""
-			(at 520 280 0)
+			(at 516.89 274.32 0)
 			(hide yes)
 			(show_name no)
@@
 		)
 		(property "Description" "Generic connector, single row, 01x02, script generated (kicad-library-utils/schlib/autogen/connector/)"
-			(at 520 280 0)
+			(at 516.89 274.32 0)
 			(hide yes)
 			(show_name no)

Commit message: more corrections and refinements before prod
Parts:
- removed R9: 1k, PCM_SparkFun-Resistor:R_0402_1005Metric, symbol PCM_SparkFun-Resistor:1k_0402
- added R12: 1k R, Resistor_SMD:R_0603_1608Metric, symbol Device:R
- R10, R11: footprint (none) -> Resistor_SMD:R_0603_1608Metric
Connections:
- net GPIO_48: now also J33.1 (Pin_1)
- net UART: now also R12.2
- net at R10.2: now also R12.1
Other:
- moved on the sheet: J33, R10
Changed lines of the file:
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@@
 	(text "TX\n"
 		(exclude_from_sim no)
-		(at 300.228 291.338 0)
+		(at 297.688 291.338 0)
 		(effects
 			(font
@@
 	)
 	(junction
+		(at 328.93 290.83)
+		(diameter 0)
+		(color 0 0 0 0)
+	)
+	(junction
 		(at 123.19 345.44)
 		(diameter 0)
@@
 	)
 	(junction
-		(at 328.93 290.83)
-		(diameter 0)
-		(color 0 0 0 0)
-	)
-	(junction
 		(at 59.69 345.44)
 		(diameter 0)
@@
 	(wire
 		(pts
-			(xy 514.92 212.54) (xy 507.3 212.54)
+			(xy 514.35 209.55) (xy 506.73 209.55)
 		)
 		(stroke
@@
 	(wire
 		(pts
-			(xy 514.92 210) (xy 507.3 210)
+			(xy 514.35 207.01) (xy 506.73 207.01)
 		)
 		(stroke
@@
 	(wire
 		(pts
+			(xy 327.66 290.83) (xy 328.93 290.83)
+		)
+		(stroke
+			(width 0)
+			(type default)
+		)
+	)
+	(wire
+		(pts
 			(xy 116.84 96.52) (xy 130.81 96.52)
 		)
@@
 	(wire
 		(pts
+			(xy 318.77 290.83) (xy 320.04 290.83)
+		)
+		(stroke
+			(width 0)
+			(type default)
+		)
+	)
+	(wire
+		(pts
 			(xy 365.08 115) (xy 372.7 115)
 		)
@@
 	(wire
 		(pts
-			(xy 312.42 290.83) (xy 313.69 290.83)
+			(xy 309.88 290.83) (xy 311.15 290.83)
 		)
 		(stroke
@@
 	(wire
 		(pts
-			(xy 322.58 290.83) (xy 321.31 290.83)
-		)
-		(stroke
-			(width 0)
-			(type default)
-		)
-	)
-	(wire
-		(pts
 			(xy 299.72 118.11) (xy 307.34 118.11)
 		)
@@
 		)
 	)
-	(wire
-		(pts
-			(xy 327.66 290.83) (xy 328.93 290.83)
-		)
-		(stroke
-			(width 0)
-			(type default)
-		)
-	)
 	(label "A1"
 		(at 514.35 41.91 180)
@@
 	(global_label "GPIO_47"
 		(shape input)
-		(at 312.42 290.83 180)
+		(at 309.88 290.83 180)
 		(effects
 			(font
@@
 		)
 		(property "Intersheetrefs" "${INTERSHEET_REFS}"
-			(at 312.42 290.83 0)
+			(at 309.88 290.83 0)
 			(hide yes)
 			(show_name no)
@@
 	(global_label "GND"
 		(shape input)
-		(at 507.3 212.54 180)
+		(at 506.73 209.55 180)
 		(effects
 			(font
@@
 		)
 		(property "Intersheetrefs" "${INTERSHEET_REFS}"
-			(at 507.3 212.54 0)
+			(at 506.73 209.55 0)
 			(hide yes)
 			(show_name no)
@@
 		)
 	)
+	(global_label "GPIO_48"
+		(shape input)
+		(at 506.73 207.01 180)
+		(effects
+			(font
+				(size 1.27 1.27)
+			)
+			(justify right)
+		)
+		(property "Intersheetrefs" "${INTERSHEET_REFS}"
+			(at 506.73 207.01 0)
+			(hide yes)
+			(show_name no)
+			(do_not_autoplace no)
+			(effects
+				(font
+					(size 1.27 1.27)
+				)
+			)
+		)
+	)
 	(global_label "MUX_CH4_SCL"
 		(shape input)
@@
 			)
 		)
-		(property "Footprint" ""
+		(property "Footprint" "Resistor_SMD:R_0603_1608Metric"
 			(at 317.5 297.688 90)
 			(hide yes)
@@
 	)
 	(symbol
-		(lib_id "PCM_SparkFun-Resistor:1k_0402")
-		(at 325.12 290.83 0)
-		(unit 1)
-		(body_style 1)
-		(exclude_from_sim no)
-		(in_bom yes)
-		(on_board yes)
-		(in_pos_files yes)
-		(dnp no)
-		(fields_autoplaced yes)
-		(property "Reference" "R9"
-			(at 325.12 284.48 0)
-			(show_name no)
-			(do_not_autoplace no)
-			(effects
-				(font
-					(size 1.27 1.27)
-				)
-			)
-		)
-		(property "Value" "1k"
-			(at 325.12 287.02 0)
-			(show_name no)
-			(do_not_autoplace no)
-			(effects
-				(font
-					(size 1.27 1.27)
-				)
-			)
-		)
-		(property "Footprint" "PCM_SparkFun-Resistor:R_0402_1005Metric"
-			(at 325.12 295.402 0)
-			(hide yes)
-			(show_name no)
-			(do_not_autoplace no)
-			(effects
-				(font
-					(size 1.27 1.27)
-				)
-			)
-		)
-		(property "Datasheet" "https://www.vishay.com/docs/20035/dcrcwe3.pdf"
-			(at 323.85 299.72 0)
-			(hide yes)
-			(show_name no)
-			(do_not_autoplace no)
-			(effects
-				(font
-					(size 1.27 1.27)
-				)
-			)
-		)
-		(property "Description" "Resistor"
-			(at 325.12 302.26 0)
-			(hide yes)
-			(show_name no)
-			(do_not_autoplace no)
-			(effects
-				(font
-					(size 1.27 1.27)
-				)
-			)
-		)
-		(property "PROD_ID" "RES-14342"
-			(at 325.12 297.688 0)
-			(hide yes)
-			(show_name no)
-			(do_not_autoplace no)
-			(effects
-				(font
-					(size 1.27 1.27)
-				)
-			)
-		)
-		(pin "2"
-		)
-		(pin "1"
-		)
-		(instances
-			(project "pantiltslide_full_turnkey"
-				(path "/069dac62-ca78-4a21-b689-b9421532705f"
-					(reference "R9")
-					(unit 1)
-				)
-			)
-		)
-	)
-	(symbol
 		(lib_id "Connector_Generic:Conn_01x03")
 		(at 437.41 170 0)
@@
 	)
 	(symbol
+		(lib_id "Device:R")
+		(at 323.85 290.83 90)
+		(unit 1)
+		(body_style 1)
+		(exclude_from_sim no)
+		(in_bom yes)
+		(on_board yes)
+		(in_pos_files yes)
+		(dnp no)
+		(property "Reference" "R12"
+			(at 323.596 288.29 90)
+			(show_name no)
+			(do_not_autoplace no)
+			(effects
+				(font
+					(size 1.27 1.27)
+				)
+			)
+		)
+		(property "Value" "1k R"
+			(at 323.85 290.83 90)
+			(show_name no)
+			(do_not_autoplace no)
+			(effects
+				(font
+					(size 1.27 1.27)
+				)
+			)
+		)
+		(property "Footprint" "Resistor_SMD:R_0603_1608Metric"
+			(at 323.85 292.608 90)
+			(hide yes)
+			(show_name no)
+			(do_not_autoplace no)
+			(effects
+				(font
+					(size 1.27 1.27)
+				)
+			)
+		)
+		(property "Datasheet" ""
+			(at 323.85 290.83 0)
+			(hide yes)
+			(show_name no)
+			(do_not_autoplace no)
+			(effects
+				(font
+					(size 1.27 1.27)
+				)
+			)
+		)
+		(property "Description" "Resistor"
+			(at 323.85 290.83 0)
+			(hide yes)
+			(show_name no)
+			(do_not_autoplace no)
+			(effects
+				(font
+					(size 1.27 1.27)
+				)
+			)
+		)
+		(pin "1"
+		)
+		(pin "2"
+		)
+		(instances
+			(project "pantiltslide_full_turnkey"
+				(path "/069dac62-ca78-4a21-b689-b9421532705f"
+					(reference "R12")
+					(unit 1)
+				)
+			)
+		)
+	)
+	(symbol
 		(lib_id "power:GND")
 		(at 144.78 382.27 0)
@@
 	(symbol
 		(lib_id "Device:R")
-		(at 317.5 290.83 90)
+		(at 314.96 290.83 90)
 		(unit 1)
 		(body_style 1)
@@
 		(dnp no)
 		(property "Reference" "R10"
-			(at 317.246 288.29 90)
+			(at 314.706 288.29 90)
 			(show_name no)
 			(do_not_autoplace no)
@@
 		)
 		(property "Value" "100R"
-			(at 317.5 290.83 90)
+			(at 314.96 290.83 90)
 			(show_name no)
 			(do_not_autoplace no)
@@
 			)
 		)
-		(property "Footprint" ""
-			(at 317.5 292.608 90)
+		(property "Footprint" "Resistor_SMD:R_0603_1608Metric"
+			(at 314.96 292.608 90)
 			(hide yes)
 			(show_name no)
@@
 		)
 		(property "Datasheet" ""
-			(at 317.5 290.83 0)
+			(at 314.96 290.83 0)
 			(hide yes)
 			(show_name no)
@@
 		)
 		(property "Description" "Resistor"
-			(at 317.5 290.83 0)
+			(at 314.96 290.83 0)
 			(hide yes)
 			(show_name no)
@@
 	(symbol
 		(lib_id "Connector_Generic:Conn_01x02")
-		(at 520 210 0)
+		(at 519.43 207.01 0)
 		(unit 1)
 		(body_style 1)
@@
 		(fields_autoplaced yes)
 		(property "Reference" "J33"
-			(at 523.24 209.9999 0)
+			(at 522.67 207.0099 0)
 			(show_name no)
 			(do_not_autoplace no)
@@
 		)
 		(property "Value" "Btn_SetKeyframe"
-			(at 523.24 212.5399 0)
+			(at 522.67 209.5499 0)
 			(show_name no)
 			(do_not_autoplace no)
@@
 		)
 		(property "Footprint" "Connector_JST:JST_XH_B2B-XH-A_1x02_P2.50mm_Vertical"
-			(at 520 210 0)
+			(at 519.43 207.01 0)
 			(hide yes)
 			(show_name no)
@@
 		)
 		(property "Datasheet" ""
-			(at 520 210 0)
+			(at 519.43 207.01 0)
 			(hide yes)
 			(show_name no)
@@
 		)
 		(property "Description" "Generic connector, single row, 01x02, script generated (kicad-library-utils/schlib/autogen/connector/)"
-			(at 520 210 0)
+			(at 519.43 207.01 0)
 			(hide yes)
 			(show_name no)
