File: pantiltslide/pantiltslide_full_turnkey_mini.kicad_pcb (KiCad board)
At the start: 4 copper layers, 54 x 93 mm, 57 parts, among them J1 Conn_01x22_Socket, J17 Motor_Slide, J2 Conn_01x22_Socket, J20 TCA9548A_Mux, J21 AS5600_Pan, J22 AS5600_Tilt, J23 OLED, J24 TCA9548A_Mux, J25 Motor_Slide, J26 Limit_Min, J27 Limit_Max, J29 Enc_Slide, J30 Enc_Pan, J31 Enc_Tilt, J32 Enc_Aux, J33 Btn_SetKeyframe, J34 ClearKeyframe, J35 Btn_PlayPause, J36 Reset, J37 5V_In, J38 24V_In, J39 Motor_Slide, J40 Motor_Slide, J41 Aux_Max, U1 tmc2209, U3 tmc2209, U5 tmc2209, U6 tmc2209

Commit message: updastes
Parts:
- moved R2 37.1 mm to (109.5, 75.2)
Routing:
- net +24V: track 0.00 -> 137.4 mm
- net SLIDE_M2B: track 0.00 -> 82.3 mm
- net SLIDE_M2A: track 0.00 -> 61.3 mm
- net SLIDE_M1B: track 0.00 -> 25.3 mm
- net SLIDE_M1A: track 0.00 -> 25.2 mm
- net Net-(J38-Pin_2): track 0.00 -> 18.2 mm
- added copper zone on B.Cu, net +24V
- added copper zone on B.Cu, net VCC_5V
