File: pantiltslide/pantiltslide_full_turnkey_mini.kicad_sch (KiCad schematic)
At the start: 63 parts, among them J1 Conn_01x22_Socket, J17 Motor_Slide, J18 Motor_Pan, J19 Motor_Tilt, J2 Conn_01x22_Socket, J20 TCA9548A_Mux, J21 AS5600_Pan, J22 AS5600_Tilt, J23 OLED, J24 TCA9548A_Mux, J26 Limit_Min, J27 Limit_Max, J28 Motor_Aux, J29 Enc_Slide, J3 MUX_2, J30 Enc_Pan, J31 Enc_Tilt, J32 Enc_Aux, J33 Btn_SetKeyframe, J34 Btn_ClearKeyframe, J35 Btn_PlayPause, J36 Btn_Reset, J37 5V_In, J38 24V_In, J4 MUX_3, J41 Aux_Max, J5 MUX_4, J6 MUX_5, J7 MUX_6, J8 MUX_7, U1 tmc2209, U2 tmc2209, U3 tmc2209, U4 tmc2209

Commit message: re wiring pcb
Connections:
- net GND: now also J3.2 (Pin_2)
Changed lines of the file:
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@@
+	(wire
+		(pts
+			(xy 539.75 68.58) (xy 560.07 68.58)
+		)
+		(stroke
+			(width 0)
+			(type default)
+		)
+	)
 	(wire
 		(pts
@@
 		)
 		(stroke
-			(width 0)
-			(type default)
-		)
-	)
-	(wire
-		(pts
-			(xy 541.02 68.58) (xy 560.07 68.58)
-		)
-		(stroke
