File: pantiltslide/pantiltslide_full_mini_extra/pantiltslide_full_mini_extra.kicad_sch (KiCad schematic)
At the start: 83 parts, among them J1 Conn_01x22_Socket, J17 Motor_Slide, J18 Motor_Pan, J19 Motor_Tilt, J2 Conn_01x22_Socket, J20 TCA9548A_Mux, J21 AS5600_Pan, J22 AS5600_Tilt, J23 OLED, J24 TCA9548A_Mux, J26 Limit_Min, J27 Limit_Max, J28 Motor_Aux, J29 Enc_Slide, J3 MUX_2, J30 Enc_Pan, J31 Enc_Tilt, J32 Enc_Aux, J33 Btn_SetKeyframe, J34 Btn_ClearKeyframe, J35 Btn_PlayPause, J36 Btn_Reset, J37 5V_In, J38 24V_In, J4 MUX_3, J41 Aux_Max, J5 MUX_4, J6 MUX_5, J7 MUX_6, J8 MUX_7, U1 tmc2209, U2 tmc2209, U3 tmc2209, U4 tmc2209

Commit message: updates
Parts:
- removed R13, R14, R15, R16, R17, R18, R19, R20, R21, R22, R23, R24: 2.2k, Resistor_SMD:R_0805_2012Metric, symbol Device:R
- F2: footprint (none) -> sww1235 KiCAD-Libraries master SW-Littelfuse:NANO-0154-OMNI-BLOK-Fuse-Holder
Connections:
- net +5V: now also C10.1, C11.1, J1.21 (Pin_21)
- removed net VCC_5V: C10.1, C11.1, F2.1, J1.21 (Pin_21), J37.2 (Pin_2)
- new net: F2.1, J37.2 (Pin_2)
Other:
- note removed: "C2-C5 belong hard against each socket's VM pin, C1 at the screw terminal."
- note removed: "Every I2C device here is a plug-in module, so these are belt-and-braces:"
- note removed: "The stepsticks carry their own VM bulk, but supply-lead inductance is what kills drivers -"
- note removed: "lift one if a module turns out to carry a strong pull-up of its own."
- moved on the sheet: C18, C19, C20, R25, R26, R27, R28
