File: pantiltslide/pantiltslide_full_mini_extra/pantiltslide_full_mini_extra.kicad_pcb (KiCad board)
At the start: 4 copper layers, 52.3 x 93.2 mm, 73 parts, among them J1 Conn_01x22_Socket, J17 Motor_Slide, J18 Motor_Pan, J19 Motor_Tilt, J2 Conn_01x22_Socket, J20 TCA9548A_Mux, J21 AS5600_Pan, J22 AS5600_Tilt, J23 OLED, J24 TCA9548A_Mux, J26 Limit_Min, J27 Limit_Max, J28 Motor_Aux, J29 Enc_Slide, J3 MUX_2, J30 Enc_Pan, J31 Enc_Tilt, J32 Enc_Aux, J33 Btn_SetKeyframe, J34 ClearKframe, J35 PlayPause, J36 Reset, J37 5V_In, J38 24V_In, J4 MUX_3, J41 Aux_Max, J5 MUX_4, J6 MUX_5, J7 MUX_6, J8 MUX_7, U1 tmc2209, U2 tmc2209, U3 tmc2209, U4 tmc2209

Commit message: formatting and spacing thing on the sch
Parts:
- J33: value Btn_SetKeyframe -> SetKframe
Routing:
- net GND: vias 13 -> 14
Other:
- board text added: "3.3v GND SDA SCL"
