File: pantiltslide/pantiltslide_full_mini_extra/pantiltslide_full_mini_extra_PROTECTION/pantiltslide_full_mini_extra_PROTECTION.kicad_pcb (KiCad board)
At the start: 4 copper layers, 52.3 x 93.2 mm, 73 parts, among them J1 Conn_01x22_Socket, J17 Motor_Slide, J18 Motor_Pan, J19 Motor_Tilt, J2 Conn_01x22_Socket, J20 TCA9548A_Mux, J21 AS5600_Pan, J22 AS5600_Tilt, J23 OLED, J24 TCA9548A_Mux, J26 Limit_Min, J27 Limit_Max, J28 Motor_Aux, J29 Enc_Slide, J3 MUX_2, J30 Enc_Pan, J31 Enc_Tilt, J32 Enc_Aux, J33 SetKframe, J34 ClearKframe, J35 PlayPause, J36 Reset, J37 5V_In, J38 24V_In, J4 MUX_3, J41 Aux_Max, J5 MUX_4, J6 MUX_5, J7 MUX_6, J8 MUX_7, U1 tmc2209, U2 tmc2209, U3 tmc2209, U4 tmc2209

Commit message: updates and new final board hopefully
Parts:
- added D1: SMBJ33A, Diode_SMD:D_SMB, B.Cu at (101.2, 106.7)
- added D2: SMBJ6.0A, Diode_SMD:D_SMB, B.Cu at (133.3, 83.7)
- added LED1: LED_24V, LED_SMD:LED_0805_2012Metric, F.Cu at (106.8, 100.6)
- added LED2: LED_5V, LED_SMD:LED_0805_2012Metric, F.Cu at (137.7, 77.7)
- added LED3: LED_3V3, LED_SMD:LED_0805_2012Metric, F.Cu at (126.0, 55.5)
- added R29: 10k, Resistor_SMD:R_0805_2012Metric, B.Cu at (88.9, 86.3)
- added R30: 10k, Resistor_SMD:R_0805_2012Metric, B.Cu at (88.9, 89.9)
- added R31: 10k, Resistor_SMD:R_0805_2012Metric, F.Cu at (106.8, 102.6)
- added R32: 2.2k, Resistor_SMD:R_0805_2012Metric, F.Cu at (137.2, 81.3)
- added R33: 1k, Resistor_SMD:R_0805_2012Metric, F.Cu at (126.0, 52.0)
- J33: value SetKframe -> Btn_SetKeyframe
- J34: value ClearKframe -> Btn_ClearKeyframe
- J35: value PlayPause -> Btn_PlayPause
- J36: value Reset -> Btn_Reset
Routing:
- net GND: track 2.54 -> 45.4 mm, vias 14 -> 15
- net +24V: track 157.1 -> 179.1 mm
- net VCC_5V: track 22.0 -> 28.1 mm, vias 0 -> 1
- net GPIO_11: track 28.9 -> 34.0 mm, vias 0 -> 1
- net 3.3v: track 423.1 -> 427.5 mm
- net GPIO_5: track 70.3 -> 72.4 mm
- net Net-(LED1-A): track 0.00 -> 2.03 mm
- net GPIO_7: track 50.4 -> 52.4 mm
- net Net-(LED2-A): track 0.00 -> 1.92 mm
- net Net-(R29-Pad2): track 0.00 -> 1.83 mm
- net Net-(LED3-A): track 0.00 -> 1.73 mm
- net MUX_CH7_SDA: track 15.9 -> 15.0 mm
