File: pantiltslide/pantiltslide_full_mini_extra/pantiltslide_full_mini_extra_PROTECTION/pantiltslide_full_mini_extra_PROTECTION.kicad_pcb (KiCad board)
At the start: 4 copper layers, 52.3 x 93.2 mm, 83 parts, among them J1 Conn_01x22_Socket, J17 Motor_Slide, J18 Motor_Pan, J19 Motor_Tilt, J2 Conn_01x22_Socket, J20 TCA9548A_Mux, J21 AS5600_Pan, J22 AS5600_Tilt, J23 OLED, J24 TCA9548A_Mux, J26 Limit_Min, J27 Limit_Max, J28 Motor_Aux, J29 Enc_Slide, J3 MUX_2, J30 Enc_Pan, J31 Enc_Tilt, J32 Enc_Aux, J33 Btn_SetKeyframe, J34 Btn_ClearKeyframe, J35 Btn_PlayPause, J36 Btn_Reset, J37 5V_In, J38 24V_In, J4 MUX_3, J41 Aux_Max, J5 MUX_4, J6 MUX_5, J7 MUX_6, J8 MUX_7, U1 tmc2209, U2 tmc2209, U3 tmc2209, U4 tmc2209

Commit message: mini_extra_PROTECTION: finalize BOM fields + layout cleanup
PCB layout (KiCad session):
- remove dangling 0.07mm VCC_5V stub near F2
- nudge F2/J37 to clear courtyard overlap
- fix J21 pad-2 GND thermal (was 1 spoke, now 2)
- zone refill; DRC now 0 errors / 0 unconnected

Schematic BOM fields:
- D1: LCSC C7427916 (NH), Manufacturer NH (was Brightking/C78419)
- D2: SMBJ6.5A, LCSC C52176732 (TDSEMIC), MPN/Mfr aligned (was SMBJ6.0A/LRC/C140903)
- F2: Value 1.5A, MPN 015401.5DR, Littelfuse, LCSC C206920
      (154 OMNI-BLOK 1.5A slow-blow Nano2 fuse+holder assembly)

Project:
- malformed_courtyard -> ignore (TMC2209 socket footprint has an
  open courtyard polygon; matches pantiltslide_full_turnkey_mini)

Still needs KiCad: Update PCB from Schematic (F8) to push the D1/D2/F2
MPN/Value/Notes fields into the board footprints (24 parity items ->
~8, remainder are the J3-J8 empty-footprint-field and REF** mounting
holes). Inner-layer copper In1 48% vs In2 55% (6.8pp) accepted -
board is only 93mm long, bow risk negligible.

Co-Authored-By: Claude Sonnet 5 <noreply@anthropic.com>
Parts:
- D2: value SMBJ6.0A -> SMBJ6.5A
- J34: value Btn_ClearKeyframe -> ClearKeyframe
- J35: value Btn_PlayPause -> PlayPause
- J36: value Btn_Reset -> Reset
- moved R31 0.27 mm to (106.8, 102.9)
- moved LED1 0.25 mm to (106.8, 100.8)
- moved F2 0.25 mm to (133.3, 84.3)
Routing:
- net GPIO_5: track 72.4 -> 70.6 mm
- net VCC_5V: track 28.1 -> 29.1 mm
Other:
- board text removed: "by AMOVFC"
Changed lines of the file:
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@@
 			(at 0 -1.65 90)
 			(layer "F.SilkS")
+			(hide yes)
 			(effects
 				(font
@@
 		(tags "LED")
 		(property "Reference" "LED2"
-			(at -0.4295 -1.524 90)
+			(at -0.762 1.524 90)
 			(layer "F.SilkS")
 			(effects
 				(font
-					(size 0.5 0.5)
+					(size 1 1)
 					(thickness 0.15)
 				)
@@
 			)
 		)
-		(property "Value" "Btn_ClearKeyframe"
-			(at 0 4.081 0)
+		(property "Value" "ClearKeyframe"
+			(at 2.032 4.081 0)
 			(layer "F.SilkS")
 			(effects
@@
 	(footprint "sww1235 KiCAD-Libraries master SW-Littelfuse:NANO-0154-OMNI-BLOK-Fuse-Holder"
 		(layer "F.Cu")
-		(at 133.35 84.582 90)
+		(at 133.34898 84.33344 90)
 		(property "Reference" "F2"
 			(at 0 0 90)
@@
 			)
 		)
-		(property "Value" "Btn_Reset"
+		(property "Value" "Reset"
 			(at 3.302 4.064 0)
 			(layer "F.SilkS")
@@
 	(footprint "Resistor_SMD:R_0805_2012Metric"
 		(layer "F.Cu")
-		(at 106.7585 102.6 180)
+		(at 106.7585 102.87 180)
 		(descr "Resistor SMD 0805 (2012 Metric), square (rectangular) end terminal, IPC-7351 nominal, (Body size source: IPC-SM-782 page 72, https://www.pcb-3d.com/wordpress/wp-content/uploads/ipc-sm-782a_amendment_1_and_2.pdf)")
 		(tags "resistor")
@@
 			(at 0 -1.65 0)
 			(layer "F.SilkS")
+			(hide yes)
 			(effects
 				(font
@@
 			(at 0 -1.65 90)
 			(layer "F.SilkS")
+			(hide yes)
 			(effects
 				(font
@@
 			)
 		)
-		(property "Value" "Btn_PlayPause"
+		(property "Value" "PlayPause"
 			(at 1.524 4.081 180)
 			(layer "F.SilkS")
@@
 	(footprint "LED_SMD:LED_0805_2012Metric"
 		(layer "F.Cu")
-		(at 106.7585 100.584)
+		(at 106.7585 100.838)
 		(descr "LED SMD 0805 (2012 Metric), square (rectangular) end terminal, IPC-7351 nominal, (Body size source: https://docs.google.com/spreadsheets/d/1BsfQQcO9C6DZCsRaXUlFlo91Tg2WpOkGARC1WS5S8t0/edit?usp=sharing)")
 		(tags "LED")
@@
 			(at 0 -1.65 0)
 			(layer "F.SilkS")
+			(hide yes)
 			(effects
 				(font
@@
 			(at 0 1.65 0)
 			(layer "F.Fab")
+			(hide yes)
 			(effects
 				(font
@@
 			(at 0 1.65 90)
 			(layer "B.SilkS")
+			(hide yes)
 			(effects
 				(font
@@
 			(at 0 1.65 90)
 			(layer "B.SilkS")
+			(hide yes)
 			(effects
 				(font
@@
 			(at 0 1.65 90)
 			(layer "B.SilkS")
+			(hide yes)
 			(effects
 				(font
@@
 			(at 0 1.65 90)
 			(layer "B.SilkS")
+			(hide yes)
 			(effects
 				(font
@@
 			)
 		)
-		(property "Value" "SMBJ6.0A"
+		(property "Value" "SMBJ6.5A"
 			(at 0 -3.1 90)
 			(layer "B.Fab")
@@
 		)
 		(property "Value" "tmc2209"
-			(at 7.366 0.598094 0)
+			(at 1.778 -14.641906 270)
+			(unlocked yes)
 			(layer "F.SilkS")
 			(effects
@@
 			(at 0 1.65 0)
 			(layer "B.SilkS")
+			(hide yes)
 			(effects
 				(font
@@
 			(at 0 1.68 0)
 			(layer "B.SilkS")
+			(hide yes)
 			(effects
 				(font
@@
 			(at -2.5875 0 90)
 			(layer "B.SilkS")
+			(hide yes)
 			(effects
 				(font
@@
 		(layer "Edge.Cuts")
 	)
-	(gr_text "v1.0"
-		(at 139.192 80.264 90)
-		(layer "F.SilkS")
-		(effects
-			(font
-				(size 0.5 0.5)
-				(thickness 0.1)
-				(bold yes)
-			)
-		)
-	)
 	(gr_text "SDA SCL"
-		(at 122.428 87.122 0)
+		(at 121.158 87.122 0)
 		(layer "F.SilkS")
 		(effects
 			(font
-				(size 0.5 0.5)
+				(size 0.8 0.8)
 				(thickness 0.125)
 				(bold yes)
@@
 	)
 	(gr_text "SDA SCL"
-		(at 122.682 99.06 0)
+		(at 121.412 99.314 0)
 		(layer "F.SilkS")
 		(effects
 			(font
-				(size 0.5 0.5)
+				(size 0.8 0.8)
 				(thickness 0.125)
 				(bold yes)
@@
 	)
 	(gr_text "SDA SCL"
-		(at 122.682 107.188 0)
+		(at 121.666 107.442 0)
 		(layer "F.SilkS")
 		(effects
 			(font
-				(size 0.5 0.5)
+				(size 0.8 0.8)
 				(thickness 0.125)
 				(bold yes)
@@
 	)
 	(gr_text "4AMP"
-		(at 99.06 105.918 0)
+		(at 98.552 104.394 0)
 		(layer "F.SilkS")
 		(effects
@@
 	)
 	(gr_text "3.3v GND SDA SCL"
-		(at 126.238 67.564 0)
+		(at 128.232 67.83 0)
 		(layer "B.SilkS")
 		(effects
 			(font
-				(size 0.5 0.5)
+				(size 0.8 0.8)
 				(thickness 0.125)
 				(bold yes)
@@
 	)
 	(gr_text "3.3v GND SDA SCL"
-		(at 126.238 74.676 0)
+		(at 128.524 74.671 0)
 		(layer "B.SilkS")
 		(effects
 			(font
-				(size 0.5 0.5)
+				(size 0.8 0.8)
 				(thickness 0.125)
 				(bold yes)
@@
 	)
 	(gr_text "GND"
-		(at 117.094 73.66 0)
+		(at 117.856 18.796 0)
 		(layer "B.SilkS")
 		(effects
@@
 	)
 	(gr_text "GND"
-		(at 117.856 18.796 0)
+		(at 118.11 70.612 0)
 		(layer "B.SilkS")
 		(effects
@@
 		)
 	)
-	(gr_text "VCC_5V"
-		(at 133.35 71.374 0)
+	(gr_text "GND"
+		(at 118.11 72.644 0)
 		(layer "B.SilkS")
 		(effects
@@
 		)
 	)
-	(gr_text "3.3v"
-		(at 133.858 19.05 0)
+	(gr_text "VCC_5V"
+		(at 133.35 71.374 0)
 		(layer "B.SilkS")
 		(effects
@@
 		)
 	)
-	(gr_text "GND"
-		(at 116.382 70.805 90)
+	(gr_text "3.3v"
+		(at 133.858 19.05 0)
 		(layer "B.SilkS")
 		(effects
@@
 		)
 	)
-	(gr_text "by AMOVFC"
-		(at 121.666 98.544 -90)
-		(layer "B.SilkS")
-		(effects
-			(font
-				(size 2.5 2.5)
-				(thickness 0.625)
-				(bold yes)
-			)
-			(justify mirror)
-		)
-	)
 	(point
 		(at 135.128 106.68)
@@
 	)
 	(segment
-		(start 134.32538 78.025)
-		(end 134.27838 77.978)
-		(width 0.2)
-		(layer "F.Cu")
-		(net "VCC_5V")
-	)
-	(segment
 		(start 133.35 81.534)
 		(end 136.5015 81.534)
@@
 	)
 	(segment
-		(start 134.27838 77.978)
+		(start 134.27838 80.21904)
 		(end 134.27838 72.136)
 		(width 2)
@@
 	)
 	(segment
-		(start 134.27838 80.46862)
-		(end 134.27838 77.978)
+		(start 133.35 81.534)
+		(end 133.35 81.397)
 		(width 2)
 		(layer "F.Cu")
@@
 	)
 	(segment
-		(start 133.35 81.534)
-		(end 133.35 81.397)
+		(start 133.34898 81.14844)
+		(end 134.27838 80.21904)
 		(width 2)
 		(layer "F.Cu")
@@
 	)
 	(segment
-		(start 137.890346 59.316)
-		(end 138.564 58.642346)
+		(start 112.268 77.724)
+		(end 116.532 73.46)
 		(width 0.2)
 		(layer "In1.Cu")
@@
 	)
 	(segment
-		(start 112.358095 80.935905)
-		(end 115.8125 77.4815)
+		(start 116.532 73.46)
+		(end 116.532 68.018)
 		(width 0.2)
 		(layer "In1.Cu")
@@
 	)
 	(segment
-		(start 110.998 80.935905)
-		(end 112.358095 80.935905)
+		(start 119.634 64.916)
+		(end 129.336314 64.916)
+		(width 0.2)
+		(layer "In1.Cu")
+		(net "GPIO_5")
+	)
+	(segment
+		(start 136.036 61.264313)
+		(end 136.036 60.217654)
 		(width 0.2)
 		(layer "In1.Cu")
@@
 	)
 	(segment
-		(start 127.87 66.382314)
-		(end 130.537001 63.715314)
+		(start 137.890346 59.316)
+		(end 138.564 58.642346)
 		(width 0.2)
 		(layer "In1.Cu")
@@
 	)
 	(segment
-		(start 136.036 61.264313)
-		(end 136.036 60.217654)
+		(start 129.336314 64.916)
+		(end 130.537 63.715314)
 		(width 0.2)
 		(layer "In1.Cu")
@@
 	)
 	(segment
-		(start 130.537001 63.715314)
-		(end 133.585 63.715314)
+		(start 136.937654 59.316)
+		(end 137.890346 59.316)
 		(width 0.2)
 		(layer "In1.Cu")
@@
 	)
 	(segment
-		(start 138.564 58.642346)
-		(end 138.564 31.376)
+		(start 133.585 63.715314)
+		(end 136.036 61.264313)
 		(width 0.2)
 		(layer "In1.Cu")
@@
 	)
 	(segment
-		(start 136.937654 59.316)
-		(end 137.890346 59.316)
+		(start 138.564 58.642346)
+		(end 138.564 31.376)
 		(width 0.2)
 		(layer "In1.Cu")
@@
 	)
 	(segment
-		(start 127.87 76.8655)
-		(end 127.87 66.382314)
+		(start 112.268 79.665905)
+		(end 112.268 77.724)
 		(width 0.2)
 		(layer "In1.Cu")
@@
 	)
 	(segment
-		(start 127.254 77.4815)
-		(end 115.8125 77.4815)
+		(start 110.998 80.935905)
+		(end 112.268 79.665905)
 		(width 0.2)
 		(layer "In1.Cu")
@@
 	)
 	(segment
-		(start 127.254 77.4815)
-		(end 127.87 76.8655)
+		(start 116.532 68.018)
+		(end 119.634 64.916)
 		(width 0.2)
 		(layer "In1.Cu")
@@
 	)
 	(segment
-		(start 133.585 63.715314)
-		(end 136.036 61.264313)
+		(start 130.537 63.715314)
+		(end 133.585 63.715314)
 		(width 0.2)
 		(layer "In1.Cu")
@@
 	)
 	(group ""
-		(members "7e52cc14-8d47-404e-a9d3-c1b58071407a" "f1f4a953-611e-4550-8f65-1deee078fd96")
+		(members "d6cf6587-8af8-4a20-ade6-a6fad9b5ce7f" "f1f4a953-611e-4550-8f65-1deee078fd96")
 	)
 	(group ""

Commit message: mini_extra_PROTECTION: sync footprint Values from schematic (F8)
Update PCB from Schematic pushed: F2 Value Fuse_Small -> 1.5A;
J34/J35/J36 button Values -> Btn_ClearKeyframe / Btn_PlayPause /
Btn_Reset. Schematic parity 24 -> 20 (remaining: D1/D2/F2 MPN and
LED/R Notes not mirrored to footprints, J3-J8 empty footprint field,
REF** mounting holes). DRC 0 errors / 0 unconnected.

Also: gitignore .history/ globally (KiCad local-history backups,
~22 MB under mini_extra).

Co-Authored-By: Claude Sonnet 5 <noreply@anthropic.com>
Parts:
- F2: value Fuse_Small -> 1.5A
- J34: value ClearKeyframe -> Btn_ClearKeyframe
- J35: value PlayPause -> Btn_PlayPause
- J36: value Reset -> Btn_Reset
Changed lines of the file:
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@@
 			)
 		)
-		(property "Value" "ClearKeyframe"
+		(property "Value" "Btn_ClearKeyframe"
 			(at 2.032 4.081 0)
 			(layer "F.SilkS")
@@
 			)
 		)
-		(property "Value" "Fuse_Small"
+		(property "Value" "1.5A"
 			(at 0 -3.429 90)
 			(layer "F.Fab")
@@
 			)
 		)
-		(property "Value" "Reset"
+		(property "Value" "Btn_Reset"
 			(at 3.302 4.064 0)
 			(layer "F.SilkS")
@@
 			)
 		)
-		(property "Value" "PlayPause"
+		(property "Value" "Btn_PlayPause"
 			(at 1.524 4.081 180)
 			(layer "F.SilkS")
