File: hardware/pantilt-controller.kicad_sch (KiCad schematic)
At the start: 81 parts, among them J1 Conn_01x22_Socket, J17 Motor_Slide, J18 Motor_Pan, J19 Motor_Tilt, J2 Conn_01x22_Socket, J20 TCA9548A_Mux, J21 AS5600_Pan, J22 AS5600_Tilt, J23 OLED, J24 TCA9548A_Mux, J26 Limit_Min, J27 Limit_Max, J28 Motor_Aux, J29 Enc_Slide, J3 MUX_2, J30 Enc_Pan, J31 Enc_Tilt, J32 Enc_Aux, J33 Btn_SetKeyframe, J34 Btn_ClearKeyframe, J35 Btn_PlayPause, J36 Btn_Reset, J37 5V_In, J38 24V_In, J4 MUX_3, J41 Aux_Max, J5 MUX_4, J6 MUX_5, J7 MUX_6, J8 MUX_7, U1 tmc2209, U2 tmc2209, U3 tmc2209, U4 tmc2209

Commit message: Split repo into hardware/ + software/, add per-area READMEs
- Move the PlatformIO firmware project (platformio.ini, src/, include/,
  docs/) into software/. Build/flash is now `cd software && pio run`.
- Move tools/pcb_review/ to hardware/tools/pcb_review/ (it reviews the
  board); update .github/workflows/pcb-review.yml paths.
- hardware/README.md: board overview, stackup, power/protection circuit,
  connector map, full BOM with verified LCSC numbers, fab notes.
  renders/ has kicad-cli 3D top+bottom images; bom.csv is the export.
- software/README.md: quick start, module map, web UI, pin map, build
  flags, bench notes. Points at docs/firmware.md for the bring-up order.
- Rewrite root README.md as an orientation doc (where hardware / software
  / legacy live) instead of duplicating the flashing guide.
- Schematic: fill in the missing LCSC part numbers for LED1-3 (C2297),
  R25-R31 (C17414), R32 (C17520), R33 (C17513 - 0805, not the 0603
  C21190); fix C1 (was a Panasonic resistor MPN -> Chengx C34642) and
  R10/R11 (-> Uniroyal C22775). Needs Update PCB from Schematic to sync.

Board unchanged electrically: ERC 0 errors, DRC 0 errors / 0 unconnected.

Co-Authored-By: Claude Sonnet 5 <noreply@anthropic.com>
Parts:
- C1: LCSC C2916286 -> C34642; MPN ERJ1HM471G16C35T -> KM477M050G20RR0VH2FP0; Manufacturer Yageo -> Chengx
- LED1, LED2, LED3: LCSC (none) -> C2297; MPN (none) -> KT-0805G; Manufacturer (none) -> Hubei KENTO
- R10, R11: LCSC C22369795 -> C22775; MPN RCA03100RFLF -> 0603WAF1000T5E; Manufacturer Royal Ohm -> Uniroyal
- R25, R26, R27, R28, R29, R30, R31: LCSC (none) -> C17414; MPN (none) -> 0805W8F1002T5E; Manufacturer (none) -> Uniroyal
- R32: LCSC (none) -> C17520; MPN (none) -> 0805W8F2201T5E; Manufacturer (none) -> Uniroyal
- R33: LCSC (none) -> C17513; MPN (none) -> 0805W8F1001T5E; Manufacturer (none) -> Uniroyal
