File: hardware/pantilt-controller.kicad_sch (KiCad schematic)
At the start: 81 parts, among them J1 Conn_01x22_Socket, J17 Motor_Slide, J18 Motor_Pan, J19 Motor_Tilt, J2 Conn_01x22_Socket, J20 TCA9548A_Mux, J21 AS5600_Pan, J22 AS5600_Tilt, J23 OLED, J24 TCA9548A_Mux, J26 Limit_Min, J27 Limit_Max, J28 Motor_Aux, J29 Enc_Slide, J3 MUX_2, J30 Enc_Pan, J31 Enc_Tilt, J32 Enc_Aux, J33 Btn_SetKeyframe, J34 Btn_ClearKeyframe, J35 Btn_PlayPause, J36 Btn_Reset, J37 5V_In, J38 24V_In, J4 MUX_3, J41 Aux_Max, J5 MUX_4, J6 MUX_5, J7 MUX_6, J8 MUX_7, U1 tmc2209, U2 tmc2209, U3 tmc2209, U4 tmc2209

Commit message: correcting fuse holder
Parts:
- F1: value Fuse -> 4A; footprint Fuse:Fuseholder_Clip-5x20mm_Littelfuse_111_Inline_P20.00x5.00mm_D1.05mm_Horizontal -> PanTilt:Fuseholder_Blade_Mini_XFCN_XF-508P-B-B; AssemblyQty 2 -> 1; LCSC C3130 -> C19727305; MPN 5x20mm PCB fuse clip -> XF-508P-B-B; Manufacturer Generic -> XFCN; Notes TWO clips per board; verify 5.00mm leg pitch -> MINI blade fuse holder XF-508P-B-B (LCSC C19727305). Footpr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
- LED1, LED2, LED3: LCSC C2297 -> C84256; MPN KT-0805G -> NCD0805R1; Manufacturer Hubei KENTO -> Nationstar
Changed lines of the file:
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@@
 			)
 		)
-		(property "Value" "Fuse"
+		(property "Value" "4A"
 			(at 56.388 24.892 90)
 			(show_name no)
@@
 			)
 		)
-		(property "Footprint" "Fuse:Fuseholder_Clip-5x20mm_Littelfuse_111_Inline_P20.00x5.00mm_D1.05mm_Horizontal"
+		(property "Footprint" "PanTilt:Fuseholder_Blade_Mini_XFCN_XF-508P-B-B"
 			(at 54.61 28.448 90)
 			(hide yes)
@@
 			)
 		)
-		(property "Description" "Fuse"
+		(property "Description" "MINI (ATM) blade fuse holder, PCB mount - 24V input protection"
 			(at 54.61 26.67 0)
 			(hide yes)
@@
 			)
 		)
-		(property "MPN" "5x20mm PCB fuse clip"
+		(property "MPN" "XF-508P-B-B"
 			(at 54.61 26.67 0)
 			(hide yes)
@@
 			)
 		)
-		(property "Manufacturer" "Generic"
+		(property "Manufacturer" "XFCN"
 			(at 54.61 26.67 0)
 			(hide yes)
@@
 			)
 		)
-		(property "LCSC" "C3130"
+		(property "LCSC" "C19727305"
 			(at 54.61 26.67 0)
 			(hide yes)
@@
 			)
 		)
-		(property "AssemblyQty" "2"
+		(property "AssemblyQty" "1"
 			(at 54.61 26.67 0)
 			(hide yes)
@@
 			)
 		)
-		(property "Notes" "TWO clips per board; verify 5.00mm leg pitch"
+		(property "Notes" "MINI blade fuse holder XF-508P-B-B (LCSC C19727305). Footprint built from XFCN drawing: 9.80 x 3.40mm hole grid, 4x 1.8mm drill (datasheet 1.6mm min; pin diagonal 1.65mm). Pad 1 = left receptacle, pad 2 = right. Takes a 4A MINI blade fuse (Littelfuse 297/997 / Bussmann ATM), ordered separately."
 			(at 54.61 26.67 0)
 			(hide yes)
@@
 			)
 		)
-		(property "MPN" "KT-0805G"
+		(property "MPN" "NCD0805R1"
 			(at 0 0 0)
 			(hide yes)
@@
 			)
 		)
-		(property "Manufacturer" "Hubei KENTO"
+		(property "Manufacturer" "Nationstar"
 			(at 0 0 0)
 			(hide yes)
@@
 			)
 		)
-		(property "LCSC" "C2297"
+		(property "LCSC" "C84256"
 			(at 0 0 0)
 			(hide yes)
@@
 			)
 		)
-		(property "MPN" "KT-0805G"
+		(property "MPN" "NCD0805R1"
 			(at 0 0 0)
 			(hide yes)
@@
 			)
 		)
-		(property "Manufacturer" "Hubei KENTO"
+		(property "Manufacturer" "Nationstar"
 			(at 0 0 0)
 			(hide yes)
@@
 			)
 		)
-		(property "LCSC" "C2297"
+		(property "LCSC" "C84256"
 			(at 0 0 0)
 			(hide yes)
@@
 			)
 		)
-		(property "MPN" "KT-0805G"
+		(property "MPN" "NCD0805R1"
 			(at 0 0 0)
 			(hide yes)
@@
 			)
 		)
-		(property "Manufacturer" "Hubei KENTO"
+		(property "Manufacturer" "Nationstar"
 			(at 0 0 0)
 			(hide yes)
@@
 			)
 		)
-		(property "LCSC" "C2297"
+		(property "LCSC" "C84256"
 			(at 0 0 0)
 			(hide yes)
