File: hardware/pantilt-controller.kicad_sch (KiCad schematic)
At the start: 81 parts, among them J1 Conn_01x22_Socket, J17 Motor_Slide, J18 Motor_Pan, J19 Motor_Tilt, J2 Conn_01x22_Socket, J20 TCA9548A_Mux, J21 AS5600_Pan, J22 AS5600_Tilt, J23 OLED, J24 TCA9548A_Mux, J26 Limit_Min, J27 Limit_Max, J28 Motor_Aux, J29 Enc_Slide, J3 MUX_2, J30 Enc_Pan, J31 Enc_Tilt, J32 Enc_Aux, J33 Btn_SetKeyframe, J34 Btn_ClearKeyframe, J35 Btn_PlayPause, J36 Btn_Reset, J37 5V_In, J38 24V_In, J4 MUX_3, J41 Aux_Max, J5 MUX_4, J6 MUX_5, J7 MUX_6, J8 MUX_7, U1 tmc2209, U2 tmc2209, U3 tmc2209, U4 tmc2209

Commit message: Document the ordered board: pin-header BOM, footprint fields, renders
Switch J23 and J3-J8 to 1x4 male pin headers (C42431787) in the schematic
and bom.csv, and give J3-J8 and U4 the footprints the PCB already has so
Update PCB from Schematic stops tripping on empty footprint fields. Refresh
both READMEs and the renders to match the board as ordered: MINI blade fuse
holder, red LEDs, pin headers, corrected top/bottom captions, and current
DRC/ERC/parity numbers.

Co-Authored-By: Claude Opus 5 <noreply@anthropic.com>
Parts:
- J23: LCSC C2718488 -> C42431787; MPN 2.54-1*4P -> PZ2.54-1X4P-H25; Manufacturer Ckmtw -> JXTCONN; Notes OLED socket -> Male 1x4 2.54mm pin header used instead of socket; same foo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
- J3, J4, J5, J6, J7, J8: footprint (none) -> Connector_PinSocket_2.54mm:PinSocket_1x04_P2.54mm_Vertical; LCSC (none) -> C42431787; MPN (none) -> PZ2.54-1X4P-H25; Manufacturer (none) -> JXTCONN; Notes (none) -> Male 1x4 2.54mm pin header used instead of socket; same foo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
- U4: footprint (none) -> TMC2209:TMC2209_SilentStepStick_Socket_18P
Changed lines of the file:
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@@
 			)
 		)
-		(property "Footprint" ""
+		(property "Footprint" "Connector_PinSocket_2.54mm:PinSocket_1x04_P2.54mm_Vertical"
 			(at 534.67 140.97 0)
 			(hide yes)
@@
 			)
 		)
+		(property "Notes" "Male 1x4 2.54mm pin header used instead of socket; same footprint copper (2.54mm pitch, 1.0mm drill)" (at 0 0 0)
+			(effects
+				(font
+					(size 1.27 1.27)
+				)
+				(hide yes)
+			)
+		)
+		(property "LCSC" "C42431787" (at 0 0 0)
+			(effects
+				(font
+					(size 1.27 1.27)
+				)
+				(hide yes)
+			)
+		)
+		(property "Manufacturer" "JXTCONN" (at 0 0 0)
+			(effects
+				(font
+					(size 1.27 1.27)
+				)
+				(hide yes)
+			)
+		)
+		(property "MPN" "PZ2.54-1X4P-H25" (at 0 0 0)
+			(effects
+				(font
+					(size 1.27 1.27)
+				)
+				(hide yes)
+			)
+		)
 		(pin "2"
 		)
@@
 			)
 		)
-		(property "Footprint" ""
+		(property "Footprint" "Connector_PinSocket_2.54mm:PinSocket_1x04_P2.54mm_Vertical"
 			(at 534.67 114.3 0)
 			(hide yes)
@@
 			)
 		)
+		(property "Notes" "Male 1x4 2.54mm pin header used instead of socket; same footprint copper (2.54mm pitch, 1.0mm drill)" (at 0 0 0)
+			(effects
+				(font
+					(size 1.27 1.27)
+				)
+				(hide yes)
+			)
+		)
+		(property "LCSC" "C42431787" (at 0 0 0)
+			(effects
+				(font
+					(size 1.27 1.27)
+				)
+				(hide yes)
+			)
+		)
+		(property "Manufacturer" "JXTCONN" (at 0 0 0)
+			(effects
+				(font
+					(size 1.27 1.27)
+				)
+				(hide yes)
+			)
+		)
+		(property "MPN" "PZ2.54-1X4P-H25" (at 0 0 0)
+			(effects
+				(font
+					(size 1.27 1.27)
+				)
+				(hide yes)
+			)
+		)
 		(pin "2"
 		)
@@
 			)
 		)
-		(property "Footprint" ""
+		(property "Footprint" "Connector_PinSocket_2.54mm:PinSocket_1x04_P2.54mm_Vertical"
 			(at 534.67 128.27 0)
 			(hide yes)
@@
 			)
 		)
+		(property "Notes" "Male 1x4 2.54mm pin header used instead of socket; same footprint copper (2.54mm pitch, 1.0mm drill)" (at 0 0 0)
+			(effects
+				(font
+					(size 1.27 1.27)
+				)
+				(hide yes)
+			)
+		)
+		(property "LCSC" "C42431787" (at 0 0 0)
+			(effects
+				(font
+					(size 1.27 1.27)
+				)
+				(hide yes)
+			)
+		)
+		(property "Manufacturer" "JXTCONN" (at 0 0 0)
+			(effects
+				(font
+					(size 1.27 1.27)
+				)
+				(hide yes)
+			)
+		)
+		(property "MPN" "PZ2.54-1X4P-H25" (at 0 0 0)
+			(effects
+				(font
+					(size 1.27 1.27)
+				)
+				(hide yes)
+			)
+		)
 		(pin "2"
 		)
@@
 			)
 		)
-		(property "Footprint" ""
+		(property "Footprint" "Connector_PinSocket_2.54mm:PinSocket_1x04_P2.54mm_Vertical"
 			(at 534.67 68.58 0)
 			(hide yes)
@@
 			)
 		)
+		(property "Notes" "Male 1x4 2.54mm pin header used instead of socket; same footprint copper (2.54mm pitch, 1.0mm drill)" (at 0 0 0)
+			(effects
+				(font
+					(size 1.27 1.27)
+				)
+				(hide yes)
+			)
+		)
+		(property "LCSC" "C42431787" (at 0 0 0)
+			(effects
+				(font
+					(size 1.27 1.27)
+				)
+				(hide yes)
+			)
+		)
+		(property "Manufacturer" "JXTCONN" (at 0 0 0)
+			(effects
+				(font
+					(size 1.27 1.27)
+				)
+				(hide yes)
+			)
+		)
+		(property "MPN" "PZ2.54-1X4P-H25" (at 0 0 0)
+			(effects
+				(font
+					(size 1.27 1.27)
+				)
+				(hide yes)
+			)
+		)
 		(pin "2"
 		)
@@
 			)
 		)
-		(property "Footprint" ""
+		(property "Footprint" "Connector_PinSocket_2.54mm:PinSocket_1x04_P2.54mm_Vertical"
 			(at 534.67 100.33 0)
 			(hide yes)
@@
 			)
 		)
+		(property "Notes" "Male 1x4 2.54mm pin header used instead of socket; same footprint copper (2.54mm pitch, 1.0mm drill)" (at 0 0 0)
+			(effects
+				(font
+					(size 1.27 1.27)
+				)
+				(hide yes)
+			)
+		)
+		(property "LCSC" "C42431787" (at 0 0 0)
+			(effects
+				(font
+					(size 1.27 1.27)
+				)
+				(hide yes)
+			)
+		)
+		(property "Manufacturer" "JXTCONN" (at 0 0 0)
+			(effects
+				(font
+					(size 1.27 1.27)
+				)
+				(hide yes)
+			)
+		)
+		(property "MPN" "PZ2.54-1X4P-H25" (at 0 0 0)
+			(effects
+				(font
+					(size 1.27 1.27)
+				)
+				(hide yes)
+			)
+		)
 		(pin "2"
 		)
@@
 			)
 		)
-		(property "MPN" "2.54-1*4P"
+		(property "MPN" "PZ2.54-1X4P-H25"
 			(at 430 120 0)
 			(hide yes)
@@
 			)
 		)
-		(property "Manufacturer" "Ckmtw"
+		(property "Manufacturer" "JXTCONN"
 			(at 430 120 0)
 			(hide yes)
@@
 			)
 		)
-		(property "LCSC" "C2718488"
+		(property "LCSC" "C42431787"
 			(at 430 120 0)
 			(hide yes)
@@
 			)
 		)
-		(property "Notes" "OLED socket"
+		(property "Notes" "Male 1x4 2.54mm pin header used instead of socket; same footprint copper (2.54mm pitch, 1.0mm drill)"
 			(at 430 120 0)
 			(hide yes)
@@
 			)
 		)
-		(property "Footprint" ""
+		(property "Footprint" "TMC2209:TMC2209_SilentStepStick_Socket_18P"
 			(at 288.29 266.7 0)
 			(hide yes)
@@
 			)
 		)
-		(property "Footprint" ""
+		(property "Footprint" "Connector_PinSocket_2.54mm:PinSocket_1x04_P2.54mm_Vertical"
 			(at 534.67 83.82 0)
 			(hide yes)
@@
 			)
 		)
+		(property "Notes" "Male 1x4 2.54mm pin header used instead of socket; same footprint copper (2.54mm pitch, 1.0mm drill)" (at 0 0 0)
+			(effects
+				(font
+					(size 1.27 1.27)
+				)
+				(hide yes)
+			)
+		)
+		(property "LCSC" "C42431787" (at 0 0 0)
+			(effects
+				(font
+					(size 1.27 1.27)
+				)
+				(hide yes)
+			)
+		)
+		(property "Manufacturer" "JXTCONN" (at 0 0 0)
+			(effects
+				(font
+					(size 1.27 1.27)
+				)
+				(hide yes)
+			)
+		)
+		(property "MPN" "PZ2.54-1X4P-H25" (at 0 0 0)
+			(effects
+				(font
+					(size 1.27 1.27)
+				)
+				(hide yes)
+			)
+		)
